File: pcb/pcb.sch (KiCad schematic (older format))
At the start: 24 parts, among them SW1 SW_Push, U1 ATmega32U4-AU, Y1 16MHz

Commit message: fix bug switches
Parts:
- MX1, MX2, MX3, MX4: footprint (none) -> MX_Alps_Hybrid:MX-1U-NoLED
Changed lines of the file:
@@
 F 0 "MX1" H 6833 3223 60  0000 C CNN
 F 1 "MX-NoLED" H 6833 3149 20  0000 C CNN
-F 2 "" H 6175 2975 60  0001 C CNN
+F 2 "MX_Alps_Hybrid:MX-1U-NoLED" H 6175 2975 60  0001 C CNN
 F 3 "" H 6175 2975 60  0001 C CNN
 	1    6800 3000
@@
 F 0 "MX2" H 7533 3223 60  0000 C CNN
 F 1 "MX-NoLED" H 7533 3149 20  0000 C CNN
-F 2 "" H 6875 2975 60  0001 C CNN
+F 2 "MX_Alps_Hybrid:MX-1U-NoLED" H 6875 2975 60  0001 C CNN
 F 3 "" H 6875 2975 60  0001 C CNN
 	1    7500 3000
@@
 F 0 "MX3" H 6833 3973 60  0000 C CNN
 F 1 "MX-NoLED" H 6833 3899 20  0000 C CNN
-F 2 "" H 6175 3725 60  0001 C CNN
+F 2 "MX_Alps_Hybrid:MX-1U-NoLED" H 6175 3725 60  0001 C CNN
 F 3 "" H 6175 3725 60  0001 C CNN
 	1    6800 3750
@@
 F 0 "MX4" H 7533 3973 60  0000 C CNN
 F 1 "MX-NoLED" H 7533 3899 20  0000 C CNN
-F 2 "" H 6875 3725 60  0001 C CNN
+F 2 "MX_Alps_Hybrid:MX-1U-NoLED" H 6875 3725 60  0001 C CNN
 F 3 "" H 6875 3725 60  0001 C CNN
 	1    7500 3750

Commit message: add usbC kicad configuration
Parts:
- removed D1, D2, D3, D4: SOD-123, Diode_SMD:D_SOD-123, symbol Device:D_Small
- removed F1: 500mA, Fuse:Fuse_1206_3216Metric, symbol Device:Polyfuse_Small
- removed MX1, MX2, MX3, MX4: MX-NoLED, MX_Alps_Hybrid:MX-1U-NoLED, symbol MX_Alps_Hybrid:MX-NoLED
- removed USB1: Molex-0548190589, random-keyboard-parts:Molex-0548190589, symbol random-keyboard-parts:Molex-0548190589
- added F1: 500mA, symbol Device:Polyfuse
- added J1: USB_C_Receptacle_USB2.0, symbol Connector:USB_C_Receptacle_USB2.0
- added R2, R5: 22, symbol Device:R_Small
- added R3, R4: 5.11k, symbol Device:R_Small
- renumbered C4 to C1, C5 to C2, C6 to C3, C7 to C4, C1 to C5, C2 to C6, C3 to C7, R2 to R6, R3 to R7, R4 to R8
Connections:
- net labels removed: COL0, COL1, ROW0, ROW1
- wire segments 63 -> 83
- no-connect marks 0 -> 2
Other:
- moved on the sheet: C1, C2, C3, C4, C5, C6, C7, R1, R6, R7, R8, SW1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

Commit message: add matrix switches
Parts:
- removed R3, R4: 5.11k, symbol Device:R_Small
- added D? (x97): 1N4148W, Diode_SMD:D_SOD-123, symbol Diode:1N4148W
- added J?: AVR-ISP-6, symbol Connector:AVR-ISP-6
- added SW? (x97): SW_Push, symbol Switch:SW_Push
Connections:
- net +5V: now also J?.2 (VCC)
- net GND: now also J?.6 (GND)
- net VCC: no longer names the net of F1.2, J1.A4 (VBUS), J1.A9 (VBUS), J1.B4 (VBUS), J1.B9 (VBUS)
- new net: D?.2 (A), SW?.2 (x97)
- new net C0: SW?.1, SW?.1, SW?.1, SW?.1, SW?.1, SW?.1, SW?.1
- new net C1: SW?.1, SW?.1, SW?.1, SW?.1, SW?.1, SW?.1
- new net C10: SW?.1, SW?.1, SW?.1, SW?.1, SW?.1, SW?.1
- new net C11: SW?.1, SW?.1, SW?.1, SW?.1, SW?.1, SW?.1
- new net C12: SW?.1, SW?.1, SW?.1, SW?.1, SW?.1, SW?.1
- new net C13: SW?.1, SW?.1, SW?.1, SW?.1, SW?.1, SW?.1
- new net C14: SW?.1, SW?.1, SW?.1, SW?.1, SW?.1, SW?.1
- new net C15: SW?.1, SW?.1, SW?.1, SW?.1, SW?.1, SW?.1
- new net C2: SW?.1, SW?.1, SW?.1, SW?.1, SW?.1, SW?.1
- new net C3: SW?.1, SW?.1, SW?.1, SW?.1, SW?.1, SW?.1
- new net C4: SW?.1, SW?.1, SW?.1, SW?.1, SW?.1, SW?.1
- new net C5: SW?.1, SW?.1, SW?.1, SW?.1, SW?.1, SW?.1
- new net C6: SW?.1, SW?.1, SW?.1, SW?.1, SW?.1, SW?.1
- new net C7: SW?.1, SW?.1, SW?.1, SW?.1, SW?.1, SW?.1
- new net C8: SW?.1, SW?.1, SW?.1, SW?.1, SW?.1, SW?.1
- new net C9: SW?.1, SW?.1, SW?.1, SW?.1, SW?.1, SW?.1
- new net R0: D?.1 (K), D?.1 (K), D?.1 (K), D?.1 (K), D?.1 (K), D?.1 (K), D?.1 (K), D?.1 (K), D?.1 (K), D?.1 (K), D?.1 (K), D?.1 (K), D?.1 (K), D?.1 (K), D?.1 (K), D?.1 (K)
- new net R1: D?.1 (K), D?.1 (K), D?.1 (K), D?.1 (K), D?.1 (K), D?.1 (K), D?.1 (K), D?.1 (K), D?.1 (K), D?.1 (K), D?.1 (K), D?.1 (K), D?.1 (K), D?.1 (K), D?.1 (K), D?.1 (K)
- new net R2: D?.1 (K), D?.1 (K), D?.1 (K), D?.1 (K), D?.1 (K), D?.1 (K), D?.1 (K), D?.1 (K), D?.1 (K), D?.1 (K), D?.1 (K), D?.1 (K), D?.1 (K), D?.1 (K), D?.1 (K), D?.1 (K)
- new net R3: D?.1 (K), D?.1 (K), D?.1 (K), D?.1 (K), D?.1 (K), D?.1 (K), D?.1 (K), D?.1 (K), D?.1 (K), D?.1 (K), D?.1 (K), D?.1 (K), D?.1 (K), D?.1 (K), D?.1 (K), D?.1 (K)
- new net R4: D?.1 (K), D?.1 (K), D?.1 (K), D?.1 (K), D?.1 (K), D?.1 (K), D?.1 (K), D?.1 (K), D?.1 (K), D?.1 (K), D?.1 (K), D?.1 (K), D?.1 (K), D?.1 (K), D?.1 (K), D?.1 (K)
- new net R5: D?.1 (K), D?.1 (K), D?.1 (K), D?.1 (K), D?.1 (K), D?.1 (K), D?.1 (K), D?.1 (K), D?.1 (K), D?.1 (K), D?.1 (K), D?.1 (K), D?.1 (K), D?.1 (K), D?.1 (K), D?.1 (K)
- new net R6: D?.1 (K)
- no-connect marks 2 -> 4
Other:
- moved on the sheet: F1

Commit message: working on pcb
Parts:
- removed D? (x81): 1N4148W, Diode_SMD:D_SOD-123, symbol Diode:1N4148W
- removed J?: AVR-ISP-6, symbol Connector:AVR-ISP-6
- removed SW? (x81): SW_Push, symbol Switch:SW_Push
- added C5: 0.1uF, Capacitor_SMD:C_0805_2012Metric, symbol Device:C_Small
- added D100, D101, D102, D103, D104, D105, D106, D107, D108, D109, D110, D111, D112, D129, D130, D131, D132, D133, D134, D135, D136, D137, D138, D139, D140, D141, D142, D143, D144, D161, D162, D163, D164, D165, D166, D167, D168, D169, D170, D171, D172, D173, D174, D175, D176, D193, D33, D34, D35, D36, D37, D38, D39, D40, D41, D42, D43, D44, D45, D46, D47, D48, D65, D66, D67, D68, D69, D70, D71, D72, D73, D74, D75, D76, D77, D78, D79, D80, D97, D98, D99: 1N4148W, Diode_SMD:D_SOD-123, symbol Diode:1N4148W
- added D113, D114, D115, D116, D117, D118, D119, D120, D121, D122, D123, D124, D125, D126, D127, D128, D145, D146, D147, D148, D149, D150, D151, D152, D153, D154, D155, D156, D157, D158, D159, D160, D17, D177, D178, D179, D18, D180, D181, D182, D183, D184, D185, D186, D187, D188, D189, D19, D190, D191, D192, D194, D20, D21, D22, D23, D24, D25, D26, D27, D28, D29, D30, D31, D32, D49, D50, D51, D52, D53, D54, D55, D56, D57, D58, D59, D60, D61, D62, D63, D64, D81, D82, D83, D84, D85, D86, D87, D88, D89, D90, D91, D92, D93, D94, D95, D96: SK6812, LED_SMD:LED_SK6812_PLCC4_5.0x5.0mm_P3.2mm, symbol LED:SK6812
- added H1, H2, H3, H4, H5, H6: MountingHole_Pad, MountingHole:MountingHole_2.5mm_Pad, symbol Mechanical:MountingHole_Pad
- added J2: ISP, Connector_PinHeader_2.54mm:PinHeader_2x03_P2.54mm_Vertical, symbol Connector_Generic:Conn_02x03_Counter_Clockwise
- added R2: 330, Resistor_SMD:R_0805_2012Metric, symbol Device:R_Small
- added SW18, SW19, SW20, SW21, SW22, SW23, SW24, SW25, SW26, SW27, SW28, SW29, SW30, SW31, SW32, SW33, SW34, SW35, SW36, SW37, SW38, SW39, SW40, SW41, SW42, SW43, SW44, SW45, SW46, SW47, SW48, SW49, SW50, SW51, SW52, SW53, SW54, SW55, SW56, SW57, SW58, SW59, SW60, SW61, SW62, SW63, SW64, SW65, SW66, SW67, SW68, SW69, SW70, SW71, SW72, SW73, SW74, SW75, SW76, SW77, SW78, SW79, SW80, SW81, SW82, SW83, SW84, SW85, SW86, SW87, SW88, SW89, SW90, SW91, SW92, SW93, SW94, SW95, SW96, SW97, SW98: SW_Push, Button_Switch_Keyboard:SW_Cherry_MX_1.00u_PCB, symbol Switch:SW_Push
- added U1: CD74HC4067M, Package_SO:SOIC-24W_7.5x15.4mm_P1.27mm, symbol 74xx:CD74HC4067M
- F1: footprint (none) -> Fuse:Fuse_1206_3216Metric
- J1: footprint (none) -> Type-C:HRO-TYPE-C-31-M-12
- R6: renamed from R2; footprint (none) -> Resistor_SMD:R_0805_2012Metric
- R7: renamed from R5; footprint (none) -> Resistor_SMD:R_0805_2012Metric
- SW1, SW10, SW11, SW12, SW13, SW14, SW15, SW16, SW2, SW3, SW4, SW5, SW6, SW7, SW8, SW9: renamed from SW?; footprint (none) -> Button_Switch_Keyboard:SW_Cherry_MX_1.00u_PCB
- SW17: renamed from SW1; footprint random-keyboard-parts:SKQG-1155865 -> Button_Switch_Keyboard:SW_Cherry_MX_1.00u_PCB
- gave numbers to parts that had none: 16
- renumbered C5 to C6, C6 to C7, C7 to C8, R6 to R3, R7 to R4, R8 to R5, U1 to U2
Connections:
- net +5V: now also C5.2, D113.3 (VDD), D114.3 (VDD), D115.3 (VDD), D116.3 (VDD), D117.3 (VDD), D118.3 (VDD), D119.3 (VDD), D120.3 (VDD), D121.3 (VDD), D122.3 (VDD), D123.3 (VDD), D124.3 (VDD), D125.3 (VDD), D126.3 (VDD), D127.3 (VDD), D128.3 (VDD), D145.3 (VDD), D146.3 (VDD), D147.3 (VDD), D148.3 (VDD), D149.3 (VDD), D150.3 (VDD), D151.3 (VDD), D152.3 (VDD), D153.3 (VDD), D154.3 (VDD), D155.3 (VDD), D156.3 (VDD), D157.3 (VDD), D158.3 (VDD), D159.3 (VDD), D160.3 (VDD), D17.3 (VDD), D177.3 (VDD), D178.3 (VDD), D179.3 (VDD), D18.3 (VDD), D180.3 (VDD), D181.3 (VDD), D182.3 (VDD), D183.3 (VDD), D184.3 (VDD), D185.3 (VDD), D186.3 (VDD), D187.3 (VDD), D188.3 (VDD), D189.3 (VDD), D19.3 (VDD), D190.3 (VDD), D191.3 (VDD), D192.3 (VDD), D194.3 (VDD), D20.3 (VDD), D21.3 (VDD), D22.3 (VDD), D23.3 (VDD), D24.3 (VDD), D25.3 (VDD), D26.3 (VDD), D27.3 (VDD), D28.3 (VDD), D29.3 (VDD), D30.3 (VDD), D31.3 (VDD), D32.3 (VDD), D49.3 (VDD), D50.3 (VDD), D51.3 (VDD), D52.3 (VDD), D53.3 (VDD), D54.3 (VDD), D55.3 (VDD), D56.3 (VDD), D57.3 (VDD), D58.3 (VDD), D59.3 (VDD), D60.3 (VDD), D61.3 (VDD), D62.3 (VDD), D63.3 (VDD), D64.3 (VDD), D81.3 (VDD), D82.3 (VDD), D83.3 (VDD), D84.3 (VDD), D85.3 (VDD), D86.3 (VDD), D87.3 (VDD), D88.3 (VDD), D89.3 (VDD), D90.3 (VDD), D91.3 (VDD), D92.3 (VDD), D93.3 (VDD), D94.3 (VDD), D95.3 (VDD), D96.3 (VDD), J2.6 (Pin_6), U1.24 (VCC)
- net C0: now also SW18.1, SW34.1, SW50.1, SW66.1, SW82.1, SW98.1, U1.9 (I0)
- net C1: now also SW19.1, SW35.1, SW51.1, SW67.1, SW83.1, U1.8 (I1)
- net C10: now also SW28.1, SW44.1, SW60.1, SW76.1, SW92.1, U1.21 (I10)
- net C11: now also SW29.1, SW45.1, SW61.1, SW77.1, SW93.1, U1.20 (I11)
- net C12: now also SW30.1, SW46.1, SW62.1, SW78.1, SW94.1, U1.19 (I12)
- net C13: now also SW31.1, SW47.1, SW63.1, SW79.1, SW95.1, U1.18 (I13)
- net C14: now also SW32.1, SW48.1, SW64.1, SW80.1, SW96.1, U1.17 (I14)
- net C15: now also SW33.1, SW49.1, SW65.1, SW81.1, SW97.1, U1.16 (I15)
- net C2: now also SW20.1, SW36.1, SW52.1, SW68.1, SW84.1, U1.7 (I2)
- net C3: now also SW21.1, SW37.1, SW53.1, SW69.1, SW85.1, U1.6 (I3)
- net C4: now also SW22.1, SW38.1, SW54.1, SW70.1, SW86.1, U1.5 (I4)
- net C5: now also SW23.1, SW39.1, SW55.1, SW71.1, SW87.1, U1.4 (I5)
- net C6: now also SW24.1, SW40.1, SW56.1, SW72.1, SW88.1, U1.3 (I6)
- net C7: now also SW25.1, SW41.1, SW57.1, SW73.1, SW89.1, U1.2 (I7)
- net C8: now also SW26.1, SW42.1, SW58.1, SW74.1, SW90.1, U1.23 (I8)
- net C9: now also SW27.1, SW43.1, SW59.1, SW75.1, SW91.1, U1.22 (I9)
- net GND: now also C5.1, D113.1 (VSS), D114.1 (VSS), D115.1 (VSS), D116.1 (VSS), D117.1 (VSS), D118.1 (VSS), D119.1 (VSS), D120.1 (VSS), D121.1 (VSS), D122.1 (VSS), D123.1 (VSS), D124.1 (VSS), D125.1 (VSS), D126.1 (VSS), D127.1 (VSS), D128.1 (VSS), D145.1 (VSS), D146.1 (VSS), D147.1 (VSS), D148.1 (VSS), D149.1 (VSS), D150.1 (VSS), D151.1 (VSS), D152.1 (VSS), D153.1 (VSS), D154.1 (VSS), D155.1 (VSS), D156.1 (VSS), D157.1 (VSS), D158.1 (VSS), D159.1 (VSS), D160.1 (VSS), D17.1 (VSS), D177.1 (VSS), D178.1 (VSS), D179.1 (VSS), D18.1 (VSS), D180.1 (VSS), D181.1 (VSS), D182.1 (VSS), D183.1 (VSS), D184.1 (VSS), D185.1 (VSS), D186.1 (VSS), D187.1 (VSS), D188.1 (VSS), D189.1 (VSS), D19.1 (VSS), D190.1 (VSS), D191.1 (VSS), D192.1 (VSS), D194.1 (VSS), D20.1 (VSS), D21.1 (VSS), D22.1 (VSS), D23.1 (VSS), D24.1 (VSS), D25.1 (VSS), D26.1 (VSS), D27.1 (VSS), D28.1 (VSS), D29.1 (VSS), D30.1 (VSS), D31.1 (VSS), D32.1 (VSS), D49.1 (VSS), D50.1 (VSS), D51.1 (VSS), D52.1 (VSS), D53.1 (VSS), D54.1 (VSS), D55.1 (VSS), D56.1 (VSS), D57.1 (VSS), D58.1 (VSS), D59.1 (VSS), D60.1 (VSS), D61.1 (VSS), D62.1 (VSS), D63.1 (VSS), D64.1 (VSS), D81.1 (VSS), D82.1 (VSS), D83.1 (VSS), D84.1 (VSS), D85.1 (VSS), D86.1 (VSS), D87.1 (VSS), D88.1 (VSS), D89.1 (VSS), D90.1 (VSS), D91.1 (VSS), D92.1 (VSS), D93.1 (VSS), D94.1 (VSS), D95.1 (VSS), D96.1 (VSS), H1.1, H2.1, H3.1, H4.1, H5.1, H6.1, J2.4 (Pin_4), U1.12 (GND)
- net R0: now also U2.41 (PF0)
- net R1: now also U2.40 (PF1), D33.1 (K), D34.1 (K), D35.1 (K), D36.1 (K), D37.1 (K), D38.1 (K), D39.1 (K), D40.1 (K), D41.1 (K), D42.1 (K), D43.1 (K), D44.1 (K), D45.1 (K), D46.1 (K), D47.1 (K), D48.1 (K)
- net R2: now also U2.39 (PF4), D65.1 (K), D66.1 (K), D67.1 (K), D68.1 (K), D69.1 (K), D70.1 (K), D71.1 (K), D72.1 (K), D73.1 (K), D74.1 (K), D75.1 (K), D76.1 (K), D77.1 (K), D78.1 (K), D79.1 (K), D80.1 (K)
- net R3: now also U2.38 (PF5), D100.1 (K), D101.1 (K), D102.1 (K), D103.1 (K), D104.1 (K), D105.1 (K), D106.1 (K), D107.1 (K), D108.1 (K), D109.1 (K), D110.1 (K), D111.1 (K), D112.1 (K), D97.1 (K), D98.1 (K), D99.1 (K)
- net R4: now also U2.37 (PF6), D129.1 (K), D130.1 (K), D131.1 (K), D132.1 (K), D133.1 (K), D134.1 (K), D135.1 (K), D136.1 (K), D137.1 (K), D138.1 (K), D139.1 (K), D140.1 (K), D141.1 (K), D142.1 (K), D143.1 (K), D144.1 (K)
- net R5: now also U2.36 (PF7), D161.1 (K), D162.1 (K), D163.1 (K), D164.1 (K), D165.1 (K), D166.1 (K), D167.1 (K), D168.1 (K), D169.1 (K), D170.1 (K), D171.1 (K), D172.1 (K), D173.1 (K), D174.1 (K), D175.1 (K), D176.1 (K)
- net R6: now also U2.31 (PC6), D193.1 (K)
- net MOSI: now reaches U2.10 (PB2)
- net MOSI: now also J2.5 (Pin_5)
- net MISO: now reaches U2.11 (PB3)
- net MISO: now also J2.1 (Pin_1)
- net LED0: now reaches U2.18 (PD0)
- net LED0: now also R2.1
- net SE: now reaches U2.25 (PD4)
- net SE: now also U1.15 (~E)
- net COM: now reaches U2.26 (PD6)
- net COM: now also U1.1 (COM)
- net S0: now reaches U2.27 (PD7)
- net S0: now also U1.10 (S0)
- net S1: now reaches U2.28 (PB4)
- net S1: now also U1.11 (S1)
- net S2: now reaches U2.29 (PB5)
- net S2: now also U1.14 (S2)
- net S3: now reaches U2.30 (PB6)
- net S3: now also U1.13 (S3)
- net SCK: now reaches U2.9 (PB1)
- net SCK: now also J2.2 (Pin_2)
- new net: D17.2 (DIN), R2.2
- new net: D17.4 (DOUT), D18.2 (DIN)
- new net: D18.4 (DOUT), D19.2 (DIN)
- new net: D19.4 (DOUT), D20.2 (DIN)
- new net: D20.4 (DOUT), D21.2 (DIN)
- new net: D21.4 (DOUT), D22.2 (DIN)
- new net: D22.4 (DOUT), D23.2 (DIN)
- new net: D23.4 (DOUT), D24.2 (DIN)
- new net: D24.4 (DOUT), D25.2 (DIN)
- new net: D25.4 (DOUT), D26.2 (DIN)
- new net: D26.4 (DOUT), D27.2 (DIN)
- new net: D27.4 (DOUT), D28.2 (DIN)
- new net: D28.4 (DOUT), D29.2 (DIN)
- new net: D29.4 (DOUT), D30.2 (DIN)
- new net: D30.4 (DOUT), D31.2 (DIN)
- new net: D31.4 (DOUT), D32.2 (DIN)
- new net: D48.2 (A), SW33.2
- new net: D47.2 (A), SW32.2
- new net: D46.2 (A), SW31.2
- new net: D45.2 (A), SW30.2
- new net: D44.2 (A), SW29.2
- new net: D43.2 (A), SW28.2
- new net: D42.2 (A), SW27.2
- new net: D41.2 (A), SW26.2
- new net: D40.2 (A), SW25.2
- new net: D39.2 (A), SW24.2
- new net: D38.2 (A), SW23.2
- new net: D37.2 (A), SW22.2
- new net: D36.2 (A), SW21.2
- new net: D35.2 (A), SW20.2
- new net: D34.2 (A), SW19.2
- new net: D33.2 (A), SW18.2
- new net: D49.4 (DOUT), D50.2 (DIN)
- new net: D50.4 (DOUT), D51.2 (DIN)
- new net: D51.4 (DOUT), D52.2 (DIN)
- new net: D52.4 (DOUT), D53.2 (DIN)
- new net: D53.4 (DOUT), D54.2 (DIN)
- new net: D54.4 (DOUT), D55.2 (DIN)
- new net: D55.4 (DOUT), D56.2 (DIN)
- new net: D56.4 (DOUT), D57.2 (DIN)
- new net: D57.4 (DOUT), D58.2 (DIN)
- new net: D58.4 (DOUT), D59.2 (DIN)
- new net: D59.4 (DOUT), D60.2 (DIN)
- new net: D60.4 (DOUT), D61.2 (DIN)
- new net: D61.4 (DOUT), D62.2 (DIN)
- new net: D62.4 (DOUT), D63.2 (DIN)
- new net: D63.4 (DOUT), D64.2 (DIN)
- new net: D80.2 (A), SW49.2
- new net: D79.2 (A), SW48.2
- new net: D78.2 (A), SW47.2
- new net: D77.2 (A), SW46.2
- new net: D76.2 (A), SW45.2
- new net: D75.2 (A), SW44.2
- new net: D74.2 (A), SW43.2
- new net: D73.2 (A), SW42.2
- new net: D72.2 (A), SW41.2
- new net: D71.2 (A), SW40.2
- new net: D70.2 (A), SW39.2
- new net: D69.2 (A), SW38.2
- new net: D68.2 (A), SW37.2
- new net: D67.2 (A), SW36.2
- new net: D66.2 (A), SW35.2
- new net: D65.2 (A), SW34.2
- new net: D81.4 (DOUT), D82.2 (DIN)
- new net: D82.4 (DOUT), D83.2 (DIN)
- new net: D83.4 (DOUT), D84.2 (DIN)
- new net: D84.4 (DOUT), D85.2 (DIN)
- new net: D85.4 (DOUT), D86.2 (DIN)
- new net: D86.4 (DOUT), D87.2 (DIN)
- new net: D87.4 (DOUT), D88.2 (DIN)
- new net: D88.4 (DOUT), D89.2 (DIN)
- new net: D89.4 (DOUT), D90.2 (DIN)
- new net: D90.4 (DOUT), D91.2 (DIN)
- new net: D91.4 (DOUT), D92.2 (DIN)
- new net: D92.4 (DOUT), D93.2 (DIN)
- new net: D93.4 (DOUT), D94.2 (DIN)
- new net: D94.4 (DOUT), D95.2 (DIN)
- new net: D95.4 (DOUT), D96.2 (DIN)
- new net: D112.2 (A), SW65.2
- new net: D111.2 (A), SW64.2
- new net: D110.2 (A), SW63.2
- new net: D109.2 (A), SW62.2
- new net: D108.2 (A), SW61.2
- new net: D107.2 (A), SW60.2
- new net: D106.2 (A), SW59.2
- new net: D105.2 (A), SW58.2
- new net: D104.2 (A), SW57.2
- new net: D103.2 (A), SW56.2
- new net: D102.2 (A), SW55.2
- new net: D101.2 (A), SW54.2
- new net: D100.2 (A), SW53.2
- new net: D99.2 (A), SW52.2
- new net: D98.2 (A), SW51.2
- new net: D97.2 (A), SW50.2
- new net: D113.4 (DOUT), D114.2 (DIN)
- new net: D114.4 (DOUT), D115.2 (DIN)
- new net: D115.4 (DOUT), D116.2 (DIN)
- new net: D116.4 (DOUT), D117.2 (DIN)
- new net: D117.4 (DOUT), D118.2 (DIN)
- new net: D118.4 (DOUT), D119.2 (DIN)
- new net: D119.4 (DOUT), D120.2 (DIN)
- new net: D120.4 (DOUT), D121.2 (DIN)
- new net: D121.4 (DOUT), D122.2 (DIN)
- new net: D122.4 (DOUT), D123.2 (DIN)
- new net: D123.4 (DOUT), D124.2 (DIN)
- new net: D124.4 (DOUT), D125.2 (DIN)
- new net: D125.4 (DOUT), D126.2 (DIN)
- new net: D126.4 (DOUT), D127.2 (DIN)
- new net: D127.4 (DOUT), D128.2 (DIN)
- new net: D144.2 (A), SW81.2
- new net: D143.2 (A), SW80.2
- new net: D142.2 (A), SW79.2
- new net: D141.2 (A), SW78.2
- new net: D140.2 (A), SW77.2
- new net: D139.2 (A), SW76.2
- new net: D138.2 (A), SW75.2
- new net: D137.2 (A), SW74.2
- new net: D136.2 (A), SW73.2
- new net: D135.2 (A), SW72.2
- new net: D134.2 (A), SW71.2
- new net: D133.2 (A), SW70.2
- new net: D132.2 (A), SW69.2
- new net: D131.2 (A), SW68.2
- new net: D130.2 (A), SW67.2
- new net: D129.2 (A), SW66.2
- new net: D145.4 (DOUT), D146.2 (DIN)
- new net: D146.4 (DOUT), D147.2 (DIN)
- new net: D147.4 (DOUT), D148.2 (DIN)
- new net: D148.4 (DOUT), D149.2 (DIN)
- new net: D149.4 (DOUT), D150.2 (DIN)
- new net: D150.4 (DOUT), D151.2 (DIN)
- new net: D151.4 (DOUT), D152.2 (DIN)
- new net: D152.4 (DOUT), D153.2 (DIN)
- new net: D153.4 (DOUT), D154.2 (DIN)
- new net: D154.4 (DOUT), D155.2 (DIN)
- new net: D155.4 (DOUT), D156.2 (DIN)
- new net: D156.4 (DOUT), D157.2 (DIN)
- new net: D157.4 (DOUT), D158.2 (DIN)
- new net: D158.4 (DOUT), D159.2 (DIN)
- new net: D159.4 (DOUT), D160.2 (DIN)
- new net: D176.2 (A), SW97.2
- new net: D175.2 (A), SW96.2
- new net: D174.2 (A), SW95.2
- new net: D173.2 (A), SW94.2
- new net: D172.2 (A), SW93.2
- new net: D171.2 (A), SW92.2
- new net: D170.2 (A), SW91.2
- new net: D169.2 (A), SW90.2
- new net: D168.2 (A), SW89.2
- new net: D167.2 (A), SW88.2
- new net: D166.2 (A), SW87.2
- new net: D165.2 (A), SW86.2
- new net: D164.2 (A), SW85.2
- new net: D163.2 (A), SW84.2
- new net: D162.2 (A), SW83.2
- new net: D161.2 (A), SW82.2
- new net: D177.4 (DOUT), D178.2 (DIN)
- new net: D178.4 (DOUT), D179.2 (DIN)
- new net: D179.4 (DOUT), D180.2 (DIN)
- new net: D180.4 (DOUT), D181.2 (DIN)
- new net: D181.4 (DOUT), D182.2 (DIN)
- new net: D182.4 (DOUT), D183.2 (DIN)
- new net: D183.4 (DOUT), D184.2 (DIN)
- new net: D184.4 (DOUT), D185.2 (DIN)
- new net: D185.4 (DOUT), D186.2 (DIN)
- new net: D186.4 (DOUT), D187.2 (DIN)
- new net: D187.4 (DOUT), D188.2 (DIN)
- new net: D188.4 (DOUT), D189.2 (DIN)
- new net: D189.4 (DOUT), D190.2 (DIN)
- new net: D190.4 (DOUT), D191.2 (DIN)
- new net: D191.4 (DOUT), D192.2 (DIN)
- new net: D193.2 (A), SW98.2
- new net LED1: D32.4 (DOUT), D49.2 (DIN)
- new net LED2: D64.4 (DOUT), D81.2 (DIN)
- new net LED3: D113.2 (DIN), D96.4 (DOUT)
- new net LED4: D128.4 (DOUT), D145.2 (DIN)
- new net LED5: D160.4 (DOUT), D177.2 (DIN)
- new net LED6: D192.4 (DOUT), D194.2 (DIN)
- new net RST: J2.3 (Pin_3)
- no-connect marks 4 -> 15
Other:
- moved on the sheet: C1, C2, C3, C4, C6, C7, C8, D1, D10, D11, D12, D13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

Commit message: sch done
Parts:
- removed Y1: 16MHz, Crystal:Crystal_SMD_3225-4Pin_3.2x2.5mm, symbol Device:Crystal_GND24_Small
- added Y1: 16MHz, Crystal:Crystal_SMD_HC49-SD, symbol Device:Crystal_Small
- H1, H2, H3, H4, H5, H6: footprint MountingHole:MountingHole_2.5mm_Pad -> MountingHole:MountingHole_2.2mm_M2_Pad_Via
- J1: footprint Type-C:HRO-TYPE-C-31-M-12 -> Connector_USB:USB_C_Receptacle_HRO_TYPE-C-31-M-12
Connections:
- net at C7.2, U2.16 (XTAL2): now also Y1.2
- net at C6.2, U2.17 (XTAL1): now also Y1.1
Other:
- moved on the sheet: C6, C7, D1, D10, D100, D101, D102, D103, D104, D105, D106, D107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

Commit message: update pcb
Parts:
- removed SW17: SW_Push, Button_Switch_Keyboard:SW_Cherry_MX_1.00u_PCB, symbol Switch:SW_Push
- SW31, SW70: footprint Button_Switch_Keyboard:SW_Cherry_MX_1.00u_PCB -> Button_Switch_Keyboard:SW_Cherry_MX_2.00u_PCB
- SW36: footprint Button_Switch_Keyboard:SW_Cherry_MX_1.00u_PCB -> Button_Switch_Keyboard:SW_Cherry_MX_1.50u_PCB
- SW49: footprint Button_Switch_Keyboard:SW_Cherry_MX_1.00u_PCB -> Button_Switch_Keyboard:SW_Cherry_MX_ISOEnter_PCB
- SW53, SW87: footprint Button_Switch_Keyboard:SW_Cherry_MX_1.00u_PCB -> Button_Switch_Keyboard:SW_Cherry_MX_2.00u_Vertical_PCB
- SW54: footprint Button_Switch_Keyboard:SW_Cherry_MX_1.00u_PCB -> Button_Switch_Keyboard:SW_Cherry_MX_1.75u_PCB
- SW91: footprint Button_Switch_Keyboard:SW_Cherry_MX_1.00u_PCB -> Button_Switch_Keyboard:SW_Cherry_MX_6.25u_PCB
Changed lines of the file:
@@
 Wire Wire Line
 	1850 2850 1850 2900
-$Comp
-L Switch:SW_Push SW17
-U 1 1 63DAF77B
-P 2100 2150
-F 0 "SW17" H 2100 2435 50  0000 C CNN
-F 1 "SW_Push" H 2100 2344 50  0000 C CNN
-F 2 "Button_Switch_Keyboard:SW_Cherry_MX_1.00u_PCB" H 2100 2350 50  0001 C CNN
-F 3 "~" H 2100 2350 50  0001 C CNN
-	1    2100 2150
-	1    0    0    -1
-$EndComp
 Wire Wire Line
 	2550 2450 2500 2450
-$Comp
-L power:GND #PWR02
-U 1 1 63DB2B3C
-P 1750 2150
-F 0 "#PWR02" H 1750 1900 50  0001 C CNN
-F 1 "GND" H 1755 1977 50  0000 C CNN
-F 2 "" H 1750 2150 50  0001 C CNN
-F 3 "" H 1750 2150 50  0001 C CNN
-	1    1750 2150
-	1    0    0    -1
-$EndComp
 Text GLabel 1850 3450 0    50   Input ~ 0
 D+
@@
 	2500 1750 3050 1750
 Wire Wire Line
-	1750 2150 1900 2150
-Wire Wire Line
-	2300 2450 2500 2450
-Wire Wire Line
-	2300 2150 2300 2450
-Connection ~ 2500 2450
-Wire Wire Line
 	2250 3250 2550 3250
 Wire Wire Line
@@
 F 0 "SW31" H 19450 4635 50  0000 C CNN
 F 1 "SW_Push" H 19450 4544 50  0000 C CNN
-F 2 "Button_Switch_Keyboard:SW_Cherry_MX_1.00u_PCB" H 19450 4550 50  0001 C CNN
+F 2 "Button_Switch_Keyboard:SW_Cherry_MX_2.00u_PCB" H 19450 4550 50  0001 C CNN
 F 3 "~" H 19450 4550 50  0001 C CNN
 	1    19450 4350
@@
 F 0 "SW49" H 20950 6385 50  0000 C CNN
 F 1 "SW_Push" H 20950 6294 50  0000 C CNN
-F 2 "Button_Switch_Keyboard:SW_Cherry_MX_1.00u_PCB" H 20950 6300 50  0001 C CNN
+F 2 "Button_Switch_Keyboard:SW_Cherry_MX_ISOEnter_PCB" H 20950 6300 50  0001 C CNN
 F 3 "~" H 20950 6300 50  0001 C CNN
 	1    20950 6100
@@
 F 0 "SW36" H 11200 6385 50  0000 C CNN
 F 1 "SW_Push" H 11200 6294 50  0000 C CNN
-F 2 "Button_Switch_Keyboard:SW_Cherry_MX_1.00u_PCB" H 11200 6300 50  0001 C CNN
+F 2 "Button_Switch_Keyboard:SW_Cherry_MX_1.50u_PCB" H 11200 6300 50  0001 C CNN
 F 3 "~" H 11200 6300 50  0001 C CNN
 	1    11200 6100
@@
 F 0 "SW54" H 12700 8035 50  0000 C CNN
 F 1 "SW_Push" H 12700 7944 50  0000 C CNN
-F 2 "Button_Switch_Keyboard:SW_Cherry_MX_1.00u_PCB" H 12700 7950 50  0001 C CNN
+F 2 "Button_Switch_Keyboard:SW_Cherry_MX_1.75u_PCB" H 12700 7950 50  0001 C CNN
 F 3 "~" H 12700 7950 50  0001 C CNN
 	1    12700 7750
@@
 F 0 "SW53" H 11950 8035 50  0000 C CNN
 F 1 "SW_Push" H 11950 7944 50  0000 C CNN
-F 2 "Button_Switch_Keyboard:SW_Cherry_MX_1.00u_PCB" H 11950 7950 50  0001 C CNN
+F 2 "Button_Switch_Keyboard:SW_Cherry_MX_2.00u_Vertical_PCB" H 11950 7950 50  0001 C CNN
 F 3 "~" H 11950 7950 50  0001 C CNN
 	1    11950 7750
@@
 F 0 "SW70" H 12700 9835 50  0000 C CNN
 F 1 "SW_Push" H 12700 9744 50  0000 C CNN
-F 2 "Button_Switch_Keyboard:SW_Cherry_MX_1.00u_PCB" H 12700 9750 50  0001 C CNN
+F 2 "Button_Switch_Keyboard:SW_Cherry_MX_2.00u_PCB" H 12700 9750 50  0001 C CNN
 F 3 "~" H 12700 9750 50  0001 C CNN
 	1    12700 9550
@@
 F 0 "SW91" H 16450 11585 50  0000 C CNN
 F 1 "SW_Push" H 16450 11494 50  0000 C CNN
-F 2 "Button_Switch_Keyboard:SW_Cherry_MX_1.00u_PCB" H 16450 11500 50  0001 C CNN
+F 2 "Button_Switch_Keyboard:SW_Cherry_MX_6.25u_PCB" H 16450 11500 50  0001 C CNN
 F 3 "~" H 16450 11500 50  0001 C CNN
 	1    16450 11300
@@
 F 0 "SW87" H 13450 11585 50  0000 C CNN
 F 1 "SW_Push" H 13450 11494 50  0000 C CNN
-F 2 "Button_Switch_Keyboard:SW_Cherry_MX_1.00u_PCB" H 13450 11500 50  0001 C CNN
+F 2 "Button_Switch_Keyboard:SW_Cherry_MX_2.00u_Vertical_PCB" H 13450 11500 50  0001 C CNN
 F 3 "~" H 13450 11500 50  0001 C CNN
 	1    13450 11300

Commit message: working on pcb
Parts:
- SW88: footprint Button_Switch_Keyboard:SW_Cherry_MX_1.00u_PCB -> Button_Switch_Keyboard:SW_Cherry_MX_1.50u_PCB
- SW94: footprint Button_Switch_Keyboard:SW_Cherry_MX_1.00u_PCB -> Button_Switch_Keyboard:SW_Cherry_MX_1.25u_PCB
Connections:
- net C1: now also SW16.1
- net C15: no longer SW16.1
- net LED1: now also D31.4 (DOUT); no longer D32.4 (DOUT)
- net R0: no longer D16.1 (K)
- net R6: now also D16.1 (K)
- net at D32.2 (DIN): now also D194.4 (DOUT); no longer D31.4 (DOUT)
Changed lines of the file:
@@
 	18150 3100 18900 3100
 Wire Wire Line
-	20400 3100 21150 3100
-Wire Wire Line
 	19650 3100 20400 3100
 Wire Wire Line
@@
 Text GLabel 21750 3100 2    50   Input ~ 0
 R0
-Wire Wire Line
-	21150 3100 21750 3100
-Connection ~ 21150 3100
-Connection ~ 20400 3100
 Connection ~ 18150 3100
 Connection ~ 17400 3100
@@
 Connection ~ 12150 3100
 Connection ~ 11400 3100
-Wire Wire Line
-	21150 3000 21150 3100
-$Comp
-L Switch:SW_Push SW16
-U 1 1 6406DE3F
-P 20950 2700
-F 0 "SW16" H 20950 2985 50  0000 C CNN
-F 1 "SW_Push" H 20950 2894 50  0000 C CNN
-F 2 "Button_Switch_Keyboard:SW_Cherry_MX_1.00u_PCB" H 20950 2900 50  0001 C CNN
-F 3 "~" H 20950 2900 50  0001 C CNN
-	1    20950 2700
-	1    0    0    -1
-$EndComp
 Text GLabel 20750 2100 1    50   Input ~ 0
 C15
-$Comp
-L Diode:1N4148W D16
-U 1 1 6406DE37
-P 21150 2850
-F 0 "D16" H 21100 3000 50  0000 C CNN
-F 1 "1N4148W" H 21100 2750 50  0000 C CNN
-F 2 "Diode_SMD:D_SOD-123" H 21150 2675 50  0001 C CNN
-F 3 "https://www.vishay.com/docs/85748/1n4148w.pdf" H 21150 2850 50  0001 C CNN
-	1    21150 2850
-	0    -1   -1   0
-$EndComp
 Wire Wire Line
 	20400 3000 20400 3100
@@
 Wire Wire Line
 	19950 3550 20100 3550
-Wire Wire Line
-	20700 3550 20850 3550
 $Comp
 L power:+5V #PWR06
@@
 Wire Wire Line
 	19650 3250 20400 3250
-Connection ~ 20400 3250
-Wire Wire Line
-	20400 3250 21150 3250
-Wire Wire Line
-	21150 3850 20400 3850
 Connection ~ 10650 3850
 Wire Wire Line
@@
 Wire Wire Line
 	19650 3850 18900 3850
-Connection ~ 20400 3850
 Wire Wire Line
 	20400 3850 19650 3850
@@
 F 0 "SW94" H 18700 11585 50  0000 C CNN
 F 1 "SW_Push" H 18700 11494 50  0000 C CNN
-F 2 "Button_Switch_Keyboard:SW_Cherry_MX_1.00u_PCB" H 18700 11500 50  0001 C CNN
+F 2 "Button_Switch_Keyboard:SW_Cherry_MX_1.25u_PCB" H 18700 11500 50  0001 C CNN
 F 3 "~" H 18700 11500 50  0001 C CNN
 	1    18700 11300
@@
 F 0 "SW88" H 14200 11585 50  0000 C CNN
 F 1 "SW_Push" H 14200 11494 50  0000 C CNN
-F 2 "Button_Switch_Keyboard:SW_Cherry_MX_1.00u_PCB" H 14200 11500 50  0001 C CNN
+F 2 "Button_Switch_Keyboard:SW_Cherry_MX_1.50u_PCB" H 14200 11500 50  0001 C CNN
 F 3 "~" H 14200 11500 50  0001 C CNN
 	1    14200 11300
@@
 	9600 12150 8950 12150
 Wire Wire Line
-	9900 13350 21750 13350
-NoConn ~ 10200 13800
-Wire Wire Line
 	8950 13800 9600 13800
 Wire Wire Line
@@
 Wire Wire Line
 	20000 9550 20000 11300
-Wire Wire Line
-	20750 2100 20750 2700
-Connection ~ 20750 2700
-Wire Wire Line
-	20750 2700 20750 4350
 Connection ~ 20750 4350
 Wire Wire Line
@@
 	1    0    0    -1
 $EndComp
-$Comp
-L LED:SK6812 D32
-U 1 1 6484D498
-P 21150 3550
-F 0 "D32" H 21400 3450 50  0000 L CNN
-F 1 "SK6812" H 21200 3800 50  0000 L CNN
-F 2 "LED_SMD:LED_SK6812_PLCC4_5.0x5.0mm_P3.2mm" H 21200 3250 50  0001 L TNN
-F 3 "https://cdn-shop.adafruit.com/product-files/1138/SK6812+LED+datasheet+.pdf" H 21250 3175 50  0001 L TNN
-	1    21150 3550
-	1    0    0    -1
-$EndComp
 Text GLabel 8950 12150 0    50   Input ~ 0
 LED5
@@
 Text GLabel 21700 5200 2    50   Input ~ 0
 LED2
-Wire Wire Line
-	21450 3550 21700 3550
 Text GLabel 21700 3550 2    50   Input ~ 0
 LED1
@@
 	0    -1   -1   0
 $EndComp
+Wire Wire Line
+	20750 2100 20750 4350
+Wire Wire Line
+	21750 3100 20400 3100
+Connection ~ 20400 3100
+Wire Wire Line
+	21700 3550 20700 3550
+Wire Wire Line
+	10650 13250 10650 13350
+$Comp
+L Switch:SW_Push SW16
+U 1 1 644B1697
+P 10450 12950
+F 0 "SW16" H 10450 13235 50  0000 C CNN
+F 1 "SW_Push" H 10450 13144 50  0000 C CNN
+F 2 "Button_Switch_Keyboard:SW_Cherry_MX_1.00u_PCB" H 10450 13150 50  0001 C CNN
+F 3 "~" H 10450 13150 50  0001 C CNN
+	1    10450 12950
+	1    0    0    -1
+$EndComp
+$Comp
+L Diode:1N4148W D16
+U 1 1 644B169D
+P 10650 13100
+F 0 "D16" H 10600 13250 50  0000 C CNN
+F 1 "1N4148W" H 10600 13000 50  0000 C CNN
+F 2 "Diode_SMD:D_SOD-123" H 10650 12925 50  0001 C CNN
+F 3 "https://www.vishay.com/docs/85748/1n4148w.pdf" H 10650 13100 50  0001 C CNN
+	1    10650 13100
+	0    -1   -1   0
+$EndComp
+$Comp
+L LED:SK6812 D32
+U 1 1 644B16A6
+P 10650 13800
+F 0 "D32" H 10900 13700 50  0000 L CNN
+F 1 "SK6812" H 10700 14050 50  0000 L CNN
+F 2 "LED_SMD:LED_SK6812_PLCC4_5.0x5.0mm_P3.2mm" H 10700 13500 50  0001 L TNN
+F 3 "https://cdn-shop.adafruit.com/product-files/1138/SK6812+LED+datasheet+.pdf" H 10750 13425 50  0001 L TNN
+	1    10650 13800
+	1    0    0    -1
+$EndComp
+Wire Wire Line
+	10250 12950 10250 11300
+Connection ~ 10250 11300
+Wire Wire Line
+	9900 13350 10650 13350
+Connection ~ 10650 13350
+Wire Wire Line
+	10650 13350 21750 13350
+Wire Wire Line
+	9900 13500 10650 13500
+Connection ~ 9900 13500
+Wire Wire Line
+	9900 14100 10650 14100
+Connection ~ 9900 14100
+Wire Wire Line
+	10200 13800 10350 13800
+NoConn ~ 10950 13800
 $EndSCHEMATC

Commit message: continue working on pcb
Connections:
- net +5V: now also C5.1; no longer C5.2
- net GND: now also C5.2, C8.1; no longer C5.1, C8.2
- net at U2.6 (UCAP): now also C8.2; no longer C8.1
Changed lines of the file:
@@
 	2150 2850 1850 2850
 Wire Wire Line
-	1850 2650 1850 2550
-Wire Wire Line
 	2150 2850 2550 2850
 Wire Wire Line
@@
 $EndComp
 $Comp
-L Device:C_Small C8
-U 1 1 63D6D4CE
-P 2250 3850
-F 0 "C8" H 2342 3896 50  0000 L CNN
-F 1 "1uF" H 2342 3805 50  0000 L CNN
-F 2 "Capacitor_SMD:C_0805_2012Metric" H 2250 3850 50  0001 C CNN
-F 3 "~" H 2250 3850 50  0001 C CNN
-	1    2250 3850
-	1    0    0    -1
-$EndComp
-$Comp
 L power:GND #PWR010
 U 1 1 63D6E1EF
@@
 $EndComp
 $Comp
-L Device:C_Small C6
-U 1 1 63D9A999
-P 1750 2550
-F 0 "C6" V 1800 2650 50  0000 C CNN
-F 1 "22uF" V 1800 2400 50  0000 C CNN
-F 2 "Capacitor_SMD:C_0805_2012Metric" H 1750 2550 50  0001 C CNN
-F 3 "~" H 1750 2550 50  0001 C CNN
-	1    1750 2550
-	0    -1   -1   0
-$EndComp
-$Comp
 L Device:C_Small C7
 U 1 1 63DA152E
@@
 Wire Wire Line
 	6000 2250 5800 2250
-$Comp
-L Device:C_Small C5
-U 1 1 6422B14C
-P 6100 2250
-F 0 "C5" V 6329 2250 50  0000 C CNN
-F 1 "0.1uF" V 6238 2250 50  0000 C CNN
-F 2 "Capacitor_SMD:C_0805_2012Metric" H 6100 2250 50  0001 C CNN
-F 3 "~" H 6100 2250 50  0001 C CNN
-	1    6100 2250
-	0    -1   -1   0
-$EndComp
 Wire Wire Line
 	16650 3100 17400 3100
@@
 	10200 13800 10350 13800
 NoConn ~ 10950 13800
+Wire Wire Line
+	1850 2650 1850 2550
+$Comp
+L Device:C_Small C6
+U 1 1 63D9A999
+P 1750 2550
+F 0 "C6" V 2000 2550 50  0000 C CNN
+F 1 "22uF" V 1900 2550 50  0000 C CNN
+F 2 "Capacitor_SMD:C_0805_2012Metric" H 1750 2550 50  0001 C CNN
+F 3 "~" H 1750 2550 50  0001 C CNN
+	1    1750 2550
+	0    -1   -1   0
+$EndComp
+$Comp
+L Device:C_Small C5
+U 1 1 6422B14C
+P 6100 2250
+F 0 "C5" V 5850 2250 50  0000 C CNN
+F 1 "0.1uF" V 5950 2250 50  0000 C CNN
+F 2 "Capacitor_SMD:C_0805_2012Metric" H 6100 2250 50  0001 C CNN
+F 3 "~" H 6100 2250 50  0001 C CNN
+	1    6100 2250
+	0    1    1    0
+$EndComp
+$Comp
+L Device:C_Small C8
+U 1 1 63D6D4CE
+P 2250 3850
+F 0 "C8" H 2000 3850 50  0000 L CNN
+F 1 "1uF" H 2000 3950 50  0000 L CNN
+F 2 "Capacitor_SMD:C_0805_2012Metric" H 2250 3850 50  0001 C CNN
+F 3 "~" H 2250 3850 50  0001 C CNN
+	1    2250 3850
+	-1   0    0    1
+$EndComp
 $EndSCHEMATC
