File: pcb/pcb.sch (KiCad schematic (older format))
At the start: 318 parts, among them J1 USB_C_Receptacle_USB2.0, J2 ISP, SW1 SW_Push, SW10 SW_Push, SW11 SW_Push, SW12 SW_Push, SW13 SW_Push, SW14 SW_Push, SW15 SW_Push, SW16 SW_Push, SW18 SW_Push, SW19 SW_Push, SW2 SW_Push, SW20 SW_Push, SW21 SW_Push, SW22 SW_Push, SW23 SW_Push, SW24 SW_Push, SW25 SW_Push, SW26 SW_Push, SW27 SW_Push, SW28 SW_Push, SW29 SW_Push, SW3 SW_Push, SW30 SW_Push, SW31 SW_Push, SW32 SW_Push, SW33 SW_Push, SW34 SW_Push, SW35 SW_Push, SW36 SW_Push, SW37 SW_Push, SW38 SW_Push, SW39 SW_Push, SW4 SW_Push, SW40 SW_Push, SW41 SW_Push, SW42 SW_Push, SW43 SW_Push, SW44 SW_Push, SW45 SW_Push, SW46 SW_Push, SW47 SW_Push, SW48 SW_Push, SW49 SW_Push, SW5 SW_Push, SW50 SW_Push, SW51 SW_Push, SW52 SW_Push, SW53 SW_Push, SW54 SW_Push, SW55 SW_Push, SW56 SW_Push, SW57 SW_Push, SW58 SW_Push, SW59 SW_Push, SW6 SW_Push, SW60 SW_Push, SW61 SW_Push, SW62 SW_Push, SW63 SW_Push, SW64 SW_Push, SW65 SW_Push, SW66 SW_Push, SW67 SW_Push, SW68 SW_Push, SW69 SW_Push, SW7 SW_Push, SW70 SW_Push, SW71 SW_Push, SW72 SW_Push, SW73 SW_Push, SW74 SW_Push, SW75 SW_Push, SW76 SW_Push, SW77 SW_Push, SW78 SW_Push, SW79 SW_Push, SW8 SW_Push, SW80 SW_Push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

Commit message: continue with pcb
Parts:
- added H7, H8, H9: MountingHole_Pad, MountingHole:MountingHole_2.2mm_M2_Pad_Via, symbol Mechanical:MountingHole_Pad
Connections:
- net GND: now also H7.1, H8.1, H9.1

Commit message: still working on it
Parts:
- added C9: 100nF, Capacitor_SMD:C_0805_2012Metric, symbol Device:C_Small
Connections:
- net GND: now also C9.2
- net at U2.42 (AREF): now also C9.1
- net RST: no longer names the net of J2.3 (Pin_3)
- no-connect marks 15 -> 16
Changed lines of the file:
@@
 NoConn ~ 6750 5550
 Wire Wire Line
-	6750 5350 7050 5350
-Wire Wire Line
 	6150 6850 6150 7000
 Connection ~ 6000 7000
@@
 Text GLabel 2950 6800 0    50   Input ~ 0
 SCK
-Text GLabel 2950 6900 0    50   Input ~ 0
-RST
 Text GLabel 3450 6800 2    50   Input ~ 0
 MOSI
@@
 P 2250 3250
 F 0 "#PWR09" H 2250 3100 50  0001 C CNN
-F 1 "+5V" H 2265 3423 50  0000 C CNN
+F 1 "+5V" H 2350 3350 50  0000 C CNN
 F 2 "" H 2250 3250 50  0001 C CNN
 F 3 "" H 2250 3250 50  0001 C CNN
@@
 Wire Wire Line
 	17400 3850 16650 3850
-Connection ~ 18150 3850
 Wire Wire Line
 	18150 3850 17400 3850
-Connection ~ 18900 3850
-Wire Wire Line
-	18900 3850 18150 3850
-Connection ~ 19650 3850
-Wire Wire Line
-	19650 3850 18900 3850
 Wire Wire Line
 	20400 3850 19650 3850
@@
 	1    0    0    -1
 $EndComp
+Wire Wire Line
+	19650 3850 18900 3850
+Connection ~ 19650 3850
+Connection ~ 18150 3850
+Connection ~ 18900 3850
+Wire Wire Line
+	18900 3850 18150 3850
+$Comp
+L Device:C_Small C9
+U 1 1 63F0ED99
+P 1300 3250
+F 0 "C9" H 1392 3296 50  0000 L CNN
+F 1 "100nF" H 1392 3205 50  0000 L CNN
+F 2 "Capacitor_SMD:C_0805_2012Metric" H 1300 3250 50  0001 C CNN
+F 3 "~" H 1300 3250 50  0001 C CNN
+	1    1300 3250
+	1    0    0    -1
+$EndComp
+$Comp
+L power:GND #PWR0102
+U 1 1 63F1653C
+P 1300 3500
+F 0 "#PWR0102" H 1300 3250 50  0001 C CNN
+F 1 "GND" H 1305 3327 50  0000 C CNN
+F 2 "" H 1300 3500 50  0001 C CNN
+F 3 "" H 1300 3500 50  0001 C CNN
+	1    1300 3500
+	1    0    0    -1
+$EndComp
+Wire Wire Line
+	1300 3500 1300 3350
+Wire Wire Line
+	1300 3150 2150 3150
+Wire Wire Line
+	2150 3150 2150 3050
+Wire Wire Line
+	2150 3050 2550 3050
+NoConn ~ 2950 6900
+Wire Wire Line
+	7050 5350 6750 5350
 $EndSCHEMATC

Commit message: near to finish pcb
Parts:
- added H10: MountingHole_Pad, MountingHole:MountingHole_2.2mm_M2_Pad_Via, symbol Mechanical:MountingHole_Pad
- SW1, SW10, SW11, SW12, SW13, SW14, SW15, SW16, SW18, SW19, SW2, SW20, SW21, SW22, SW23, SW24, SW25, SW26, SW27, SW28, SW29, SW3, SW30, SW32, SW33, SW34, SW35, SW37, SW38, SW39, SW4, SW40, SW41, SW42, SW43, SW44, SW45, SW46, SW47, SW48, SW5, SW50, SW51, SW52, SW55, SW56, SW57, SW58, SW59, SW6, SW60, SW61, SW62, SW63, SW64, SW65, SW66, SW67, SW68, SW69, SW7, SW71, SW72, SW73, SW74, SW75, SW76, SW77, SW78, SW79, SW8, SW80, SW81, SW82, SW83, SW84, SW85, SW86, SW89, SW9, SW90, SW92, SW93, SW95, SW96, SW97, SW98: footprint Button_Switch_Keyboard:SW_Cherry_MX_1.00u_PCB -> Button_Switch_Keyboard:SW_Cherry_MX_1.00u_Plate
- SW36, SW88: footprint Button_Switch_Keyboard:SW_Cherry_MX_1.50u_PCB -> Button_Switch_Keyboard:SW_Cherry_MX_1.50u_Plate
- SW54: footprint Button_Switch_Keyboard:SW_Cherry_MX_1.75u_PCB -> Button_Switch_Keyboard:SW_Cherry_MX_1.00u_Plate
- SW94: footprint Button_Switch_Keyboard:SW_Cherry_MX_1.25u_PCB -> Button_Switch_Keyboard:SW_Cherry_MX_1.25u_Plate
Connections:
- net GND: now also H10.1
Other:
- moved on the sheet: F1

Commit message: near to have final version pcb ;)
Parts:
- SW54: footprint Button_Switch_Keyboard:SW_Cherry_MX_1.00u_Plate -> Button_Switch_Keyboard:SW_Cherry_MX_1.75u_Plate
Changed lines of the file:
@@
 F 0 "SW54" H 12700 8035 50  0000 C CNN
 F 1 "SW_Push" H 12700 7944 50  0000 C CNN
-F 2 "Button_Switch_Keyboard:SW_Cherry_MX_1.00u_Plate" H 12700 7950 50  0001 C CNN
+F 2 "Button_Switch_Keyboard:SW_Cherry_MX_1.75u_Plate" H 12700 7950 50  0001 C CNN
 F 3 "~" H 12700 7950 50  0001 C CNN
 	1    12700 7750

Commit message: add test pcb
Parts:
- C1, C2, C3, C4, C5, C6, C7, C8, C9: footprint Capacitor_SMD:C_0805_2012Metric -> Capacitor_SMD:C_1206_3216Metric
- R1, R2, R3, R4, R5, R6, R7: footprint Resistor_SMD:R_0805_2012Metric -> Resistor_SMD:R_1206_3216Metric
Changed lines of the file:
@@
 F 0 "R7" V 7100 6100 50  0000 C CNN
 F 1 "22" V 7200 6100 50  0000 C CNN
-F 2 "Resistor_SMD:R_0805_2012Metric" H 7000 6100 50  0001 C CNN
+F 2 "Resistor_SMD:R_1206_3216Metric" H 7000 6100 50  0001 C CNN
 F 3 "~" H 7000 6100 50  0001 C CNN
 	1    7000 6100
@@
 F 0 "R6" V 6804 5900 50  0000 C CNN
 F 1 "22" V 6895 5900 50  0000 C CNN
-F 2 "Resistor_SMD:R_0805_2012Metric" H 7000 5900 50  0001 C CNN
+F 2 "Resistor_SMD:R_1206_3216Metric" H 7000 5900 50  0001 C CNN
 F 3 "~" H 7000 5900 50  0001 C CNN
 	1    7000 5900
@@
 F 0 "R5" V 4004 4550 50  0000 C CNN
 F 1 "10k" V 4095 4550 50  0000 C CNN
-F 2 "Resistor_SMD:R_0805_2012Metric" H 4200 4550 50  0001 C CNN
+F 2 "Resistor_SMD:R_1206_3216Metric" H 4200 4550 50  0001 C CNN
 F 3 "~" H 4200 4550 50  0001 C CNN
 	1    4200 4550
@@
 F 0 "R3" V 1904 3450 50  0000 C CNN
 F 1 "22" V 1995 3450 50  0000 C CNN
-F 2 "Resistor_SMD:R_0805_2012Metric" H 2100 3450 50  0001 C CNN
+F 2 "Resistor_SMD:R_1206_3216Metric" H 2100 3450 50  0001 C CNN
 F 3 "~" H 2100 3450 50  0001 C CNN
 	1    2100 3450
@@
 F 0 "R4" V 2200 3550 50  0000 C CNN
 F 1 "22" V 2300 3550 50  0000 C CNN
-F 2 "Resistor_SMD:R_0805_2012Metric" H 2100 3550 50  0001 C CNN
+F 2 "Resistor_SMD:R_1206_3216Metric" H 2100 3550 50  0001 C CNN
 F 3 "~" H 2100 3550 50  0001 C CNN
 	1    2100 3550
@@
 F 0 "C7" V 1650 3000 50  0000 C CNN
 F 1 "22uF" V 1650 2750 50  0000 C CNN
-F 2 "Capacitor_SMD:C_0805_2012Metric" H 1750 2900 50  0001 C CNN
+F 2 "Capacitor_SMD:C_1206_3216Metric" H 1750 2900 50  0001 C CNN
 F 3 "~" H 1750 2900 50  0001 C CNN
 	1    1750 2900
@@
 F 0 "C2" H 3942 2046 50  0000 L CNN
 F 1 "0.1uF" H 3942 1955 50  0000 L CNN
-F 2 "Capacitor_SMD:C_0805_2012Metric" H 3850 2000 50  0001 C CNN
+F 2 "Capacitor_SMD:C_1206_3216Metric" H 3850 2000 50  0001 C CNN
 F 3 "~" H 3850 2000 50  0001 C CNN
 	1    3850 2000
@@
 F 0 "C3" H 4342 2046 50  0000 L CNN
 F 1 "0.1uF" H 4342 1955 50  0000 L CNN
-F 2 "Capacitor_SMD:C_0805_2012Metric" H 4250 2000 50  0001 C CNN
+F 2 "Capacitor_SMD:C_1206_3216Metric" H 4250 2000 50  0001 C CNN
 F 3 "~" H 4250 2000 50  0001 C CNN
 	1    4250 2000
@@
 F 0 "C4" H 4742 2046 50  0000 L CNN
 F 1 "10uF" H 4742 1955 50  0000 L CNN
-F 2 "Capacitor_SMD:C_0805_2012Metric" H 4650 2000 50  0001 C CNN
+F 2 "Capacitor_SMD:C_1206_3216Metric" H 4650 2000 50  0001 C CNN
 F 3 "~" H 4650 2000 50  0001 C CNN
 	1    4650 2000
@@
 F 0 "C1" H 3542 2046 50  0000 L CNN
 F 1 "0.1uF" H 3542 1955 50  0000 L CNN
-F 2 "Capacitor_SMD:C_0805_2012Metric" H 3450 2000 50  0001 C CNN
+F 2 "Capacitor_SMD:C_1206_3216Metric" H 3450 2000 50  0001 C CNN
 F 3 "~" H 3450 2000 50  0001 C CNN
 	1    3450 2000
@@
 F 0 "R1" H 2559 2096 50  0000 L CNN
 F 1 "10k" H 2559 2005 50  0000 L CNN
-F 2 "Resistor_SMD:R_0805_2012Metric" H 2500 2050 50  0001 C CNN
+F 2 "Resistor_SMD:R_1206_3216Metric" H 2500 2050 50  0001 C CNN
 F 3 "~" H 2500 2050 50  0001 C CNN
 	1    2500 2050
@@
 F 0 "R2" V 9396 3550 50  0000 C CNN
 F 1 "330" V 9305 3550 50  0000 C CNN
-F 2 "Resistor_SMD:R_0805_2012Metric" H 9200 3550 50  0001 C CNN
+F 2 "Resistor_SMD:R_1206_3216Metric" H 9200 3550 50  0001 C CNN
 F 3 "~" H 9200 3550 50  0001 C CNN
 	1    9200 3550
@@
 F 0 "C6" V 2000 2550 50  0000 C CNN
 F 1 "22uF" V 1900 2550 50  0000 C CNN
-F 2 "Capacitor_SMD:C_0805_2012Metric" H 1750 2550 50  0001 C CNN
+F 2 "Capacitor_SMD:C_1206_3216Metric" H 1750 2550 50  0001 C CNN
 F 3 "~" H 1750 2550 50  0001 C CNN
 	1    1750 2550
@@
 F 0 "C5" V 5850 2250 50  0000 C CNN
 F 1 "0.1uF" V 5950 2250 50  0000 C CNN
-F 2 "Capacitor_SMD:C_0805_2012Metric" H 6100 2250 50  0001 C CNN
+F 2 "Capacitor_SMD:C_1206_3216Metric" H 6100 2250 50  0001 C CNN
 F 3 "~" H 6100 2250 50  0001 C CNN
 	1    6100 2250
@@
 F 0 "C8" H 2000 3850 50  0000 L CNN
 F 1 "1uF" H 2000 3950 50  0000 L CNN
-F 2 "Capacitor_SMD:C_0805_2012Metric" H 2250 3850 50  0001 C CNN
+F 2 "Capacitor_SMD:C_1206_3216Metric" H 2250 3850 50  0001 C CNN
 F 3 "~" H 2250 3850 50  0001 C CNN
 	1    2250 3850
@@
 F 0 "C9" H 1392 3296 50  0000 L CNN
 F 1 "100nF" H 1392 3205 50  0000 L CNN
-F 2 "Capacitor_SMD:C_0805_2012Metric" H 1300 3250 50  0001 C CNN
+F 2 "Capacitor_SMD:C_1206_3216Metric" H 1300 3250 50  0001 C CNN
 F 3 "~" H 1300 3250 50  0001 C CNN
 	1    1300 3250

Commit message: update budget
Parts:
- C9: value 100nF -> 0.1uF
Changed lines of the file:
@@
 P 1300 3250
 F 0 "C9" H 1392 3296 50  0000 L CNN
-F 1 "100nF" H 1392 3205 50  0000 L CNN
+F 1 "0.1uF" H 1392 3205 50  0000 L CNN
 F 2 "Capacitor_SMD:C_1206_3216Metric" H 1300 3250 50  0001 C CNN
 F 3 "~" H 1300 3250 50  0001 C CNN
