File: pcb/pcb.kicad_pcb (KiCad board)
At the start: 2 copper layers, 24 parts, among them SW1 SW_Push, U1 ATmega32U4-AU, Y1 16MHz

Commit message: working on pcb
Parts:
- removed C1, C2: 22uF, Capacitor_SMD:C_0805_2012Metric
- removed C3: 1uF, Capacitor_SMD:C_0805_2012Metric
- removed C4, C5, C6: 0.1uF, Capacitor_SMD:C_0805_2012Metric
- removed C7: 10uF, Capacitor_SMD:C_0805_2012Metric
- removed D1, D2, D3, D4: SOD-123, Diode_SMD:D_SOD-123
- removed F1: 500mA, Fuse:Fuse_1206_3216Metric
- removed MX1, MX2, MX3, MX4: MX-NoLED, MX_Alps_Hybrid:MX-1U-NoLED
- removed R1, R4: 10k, Resistor_SMD:R_0805_2012Metric
- removed R2, R3: 22, Resistor_SMD:R_0805_2012Metric
- removed SW1: SW_Push, random-keyboard-parts:SKQG-1155865
- removed U1: ATmega32U4-AU, Package_QFP:TQFP-44_10x10mm_P0.8mm
- removed USB1: Molex-0548190589, random-keyboard-parts:Molex-0548190589
- removed Y1: 16MHz, Crystal:Crystal_SMD_3225-4Pin_3.2x2.5mm

Commit message: update pcb
Parts:
- added C1: 0.1uF, Capacitor_SMD:C_0805_2012Metric, F.Cu at (167.9, -198.8)
- added C2: 0.1uF, Capacitor_SMD:C_0805_2012Metric, F.Cu at (225.0, -218.6)
- added C3: 0.1uF, Capacitor_SMD:C_0805_2012Metric, F.Cu at (197.0, -191.8)
- added C4: 10uF, Capacitor_SMD:C_0805_2012Metric, F.Cu at (172.3, -198.8)
- added C5: 0.1uF, Capacitor_SMD:C_0805_2012Metric, F.Cu at (353.9, -370.1)
- added C6: 22uF, Capacitor_SMD:C_0805_2012Metric, F.Cu at (353.9, -365.7)
- added C7: 22uF, Capacitor_SMD:C_0805_2012Metric, F.Cu at (349.0, -374.8)
- added C8: 1uF, Capacitor_SMD:C_0805_2012Metric, F.Cu at (349.0, -370.4)
- added D1: 1N4148W, Diode_SMD:D_SOD-123, B.Cu at (17.8, -365.6)
- added D10: 1N4148W, Diode_SMD:D_SOD-123, B.Cu at (189.2, -365.6)
- added D100: 1N4148W, Diode_SMD:D_SOD-123, B.Cu at (360.7, -317.6)
- added D101: 1N4148W, Diode_SMD:D_SOD-123, F.Cu at (171.4, -205.3)
- added D102: 1N4148W, Diode_SMD:D_SOD-123, F.Cu at (203.7, -204.9)
- added D103: 1N4148W, Diode_SMD:D_SOD-123, F.Cu at (322.7, -189.5)
- added D104: 1N4148W, Diode_SMD:D_SOD-123, F.Cu at (345.5, -213.0)
- added D105: 1N4148W, Diode_SMD:D_SOD-123, F.Cu at (339.5, -207.1)
- added D106: 1N4148W, Diode_SMD:D_SOD-123, F.Cu at (223.9, -228.4)
- added D107: 1N4148W, Diode_SMD:D_SOD-123, F.Cu at (203.7, -208.2)
- added D108: 1N4148W, Diode_SMD:D_SOD-123, F.Cu at (179.8, -215.6)
- added D109: 1N4148W, Diode_SMD:D_SOD-123, F.Cu at (212.1, -215.1)
- added D11: 1N4148W, Diode_SMD:D_SOD-123, B.Cu at (208.3, -365.6)
- added D110: 1N4148W, Diode_SMD:D_SOD-123, F.Cu at (215.5, -221.8)
- added D111: 1N4148W, Diode_SMD:D_SOD-123, F.Cu at (179.8, -212.2)
- added D112: 1N4148W, Diode_SMD:D_SOD-123, F.Cu at (36.7, -205.5)
- added D113: SK6812, LED_SMD:LED_SK6812_PLCC4_5.0x5.0mm_P3.2mm, F.Cu at (295.3, -338.5)
- added D114: SK6812, LED_SMD:LED_SK6812_PLCC4_5.0x5.0mm_P3.2mm, F.Cu at (314.5, -338.5)
- added D115: SK6812, LED_SMD:LED_SK6812_PLCC4_5.0x5.0mm_P3.2mm, F.Cu at (333.4, -338.5)
- added D116: SK6812, LED_SMD:LED_SK6812_PLCC4_5.0x5.0mm_P3.2mm, F.Cu at (352.4, -328.9)
- added D117: SK6812, LED_SMD:LED_SK6812_PLCC4_5.0x5.0mm_P3.2mm, F.Cu at (155.9, -207.0)
- added D118: SK6812, LED_SMD:LED_SK6812_PLCC4_5.0x5.0mm_P3.2mm, F.Cu at (335.8, -231.3)
- added D119: SK6812, LED_SMD:LED_SK6812_PLCC4_5.0x5.0mm_P3.2mm, F.Cu at (177.8, -227.2)
- added D12: 1N4148W, Diode_SMD:D_SOD-123, B.Cu at (227.3, -365.6)
- added D120: SK6812, LED_SMD:LED_SK6812_PLCC4_5.0x5.0mm_P3.2mm, F.Cu at (295.4, -183.9)
- added D121: SK6812, LED_SMD:LED_SK6812_PLCC4_5.0x5.0mm_P3.2mm, F.Cu at (275.2, -163.7)
- added D122: SK6812, LED_SMD:LED_SK6812_PLCC4_5.0x5.0mm_P3.2mm, F.Cu at (315.6, -197.8)
- added D123: SK6812, LED_SMD:LED_SK6812_PLCC4_5.0x5.0mm_P3.2mm, F.Cu at (208.4, -233.4)
- added D124: SK6812, LED_SMD:LED_SK6812_PLCC4_5.0x5.0mm_P3.2mm, F.Cu at (188.2, -213.2)
- added D125: SK6812, LED_SMD:LED_SK6812_PLCC4_5.0x5.0mm_P3.2mm, F.Cu at (315.6, -204.4)
- added D126: SK6812, LED_SMD:LED_SK6812_PLCC4_5.0x5.0mm_P3.2mm, F.Cu at (155.9, -213.6)
- added D127: SK6812, LED_SMD:LED_SK6812_PLCC4_5.0x5.0mm_P3.2mm, F.Cu at (147.4, -207.0)
- added D128: SK6812, LED_SMD:LED_SK6812_PLCC4_5.0x5.0mm_P3.2mm, F.Cu at (147.4, -213.6)
- added D129: 1N4148W, Diode_SMD:D_SOD-123, F.Cu at (227.0, -221.7)
- added D13: 1N4148W, Diode_SMD:D_SOD-123, B.Cu at (246.4, -365.6)
- added D130: 1N4148W, Diode_SMD:D_SOD-123, F.Cu at (195.0, -188.3)
- added D131: 1N4148W, Diode_SMD:D_SOD-123, F.Cu at (322.4, -179.4)
- added D132: 1N4148W, Diode_SMD:D_SOD-123, F.Cu at (203.4, -201.5)
- added D133: 1N4148W, Diode_SMD:D_SOD-123, F.Cu at (290.7, -156.0)
- added D134: 1N4148W, Diode_SMD:D_SOD-123, F.Cu at (296.7, -162.3)
- added D135: 1N4148W, Diode_SMD:D_SOD-123, F.Cu at (310.9, -176.2)
- added D136: 1N4148W, Diode_SMD:D_SOD-123, F.Cu at (316.9, -182.9)
- added D137: 1N4148W, Diode_SMD:D_SOD-123, F.Cu at (193.3, -225.5)
- added D138: 1N4148W, Diode_SMD:D_SOD-123, F.Cu at (189.3, -188.0)
- added D139: 1N4148W, Diode_SMD:D_SOD-123, F.Cu at (232.3, -235.3)
- added D14: 1N4148W, Diode_SMD:D_SOD-123, B.Cu at (265.4, -365.6)
- added D140: 1N4148W, Diode_SMD:D_SOD-123, F.Cu at (19.2, -200.8)
- added D141: 1N4148W, Diode_SMD:D_SOD-123, F.Cu at (322.7, -192.8)
- added D142: 1N4148W, Diode_SMD:D_SOD-123, F.Cu at (183.5, -188.0)
- added D143: 1N4148W, Diode_SMD:D_SOD-123, F.Cu at (30.7, -200.8)
- added D144: 1N4148W, Diode_SMD:D_SOD-123, F.Cu at (25.0, -200.8)
- added D145: SK6812, LED_SMD:LED_SK6812_PLCC4_5.0x5.0mm_P3.2mm, F.Cu at (130.6, -207.0)
- added D146: SK6812, LED_SMD:LED_SK6812_PLCC4_5.0x5.0mm_P3.2mm, F.Cu at (130.6, -213.6)
- added D147: SK6812, LED_SMD:LED_SK6812_PLCC4_5.0x5.0mm_P3.2mm, F.Cu at (122.2, -207.0)
- added D148: SK6812, LED_SMD:LED_SK6812_PLCC4_5.0x5.0mm_P3.2mm, F.Cu at (335.8, -237.9)
- added D149: SK6812, LED_SMD:LED_SK6812_PLCC4_5.0x5.0mm_P3.2mm, F.Cu at (324.0, -204.4)
- added D15: 1N4148W, Diode_SMD:D_SOD-123, B.Cu at (284.5, -365.6)
- added D150: SK6812, LED_SMD:LED_SK6812_PLCC4_5.0x5.0mm_P3.2mm, F.Cu at (176.4, -193.0)
- added D151: SK6812, LED_SMD:LED_SK6812_PLCC4_5.0x5.0mm_P3.2mm, F.Cu at (324.0, -211.1)
- added D152: SK6812, LED_SMD:LED_SK6812_PLCC4_5.0x5.0mm_P3.2mm, F.Cu at (196.6, -213.2)
- added D153: SK6812, LED_SMD:LED_SK6812_PLCC4_5.0x5.0mm_P3.2mm, F.Cu at (332.4, -204.4)
- added D154: SK6812, LED_SMD:LED_SK6812_PLCC4_5.0x5.0mm_P3.2mm, F.Cu at (283.6, -157.1)
- added D155: SK6812, LED_SMD:LED_SK6812_PLCC4_5.0x5.0mm_P3.2mm, F.Cu at (216.8, -226.8)
- added D156: SK6812, LED_SMD:LED_SK6812_PLCC4_5.0x5.0mm_P3.2mm, F.Cu at (205.0, -213.2)
- added D157: SK6812, LED_SMD:LED_SK6812_PLCC4_5.0x5.0mm_P3.2mm, F.Cu at (225.2, -233.4)
- added D158: SK6812, LED_SMD:LED_SK6812_PLCC4_5.0x5.0mm_P3.2mm, F.Cu at (184.8, -193.0)
- added D159: SK6812, LED_SMD:LED_SK6812_PLCC4_5.0x5.0mm_P3.2mm, F.Cu at (324.0, -197.8)
- added D16: 1N4148W, Diode_SMD:D_SOD-123, F.Cu at (308.2, -165.6)
- added D160: SK6812, LED_SMD:LED_SK6812_PLCC4_5.0x5.0mm_P3.2mm, F.Cu at (295.4, -170.7)
- added D161: 1N4148W, Diode_SMD:D_SOD-123, F.Cu at (316.9, -186.2)
- added D162: 1N4148W, Diode_SMD:D_SOD-123, F.Cu at (195.3, -201.6)
- added D163: 1N4148W, Diode_SMD:D_SOD-123, F.Cu at (296.7, -165.7)
- added D164: 1N4148W, Diode_SMD:D_SOD-123, F.Cu at (290.7, -159.4)
- added D165: 1N4148W, Diode_SMD:D_SOD-123, F.Cu at (171.4, -208.6)
- added D166: 1N4148W, Diode_SMD:D_SOD-123, F.Cu at (163.0, -202.0)
- added D167: 1N4148W, Diode_SMD:D_SOD-123, F.Cu at (334.2, -192.8)
- added D168: 1N4148W, Diode_SMD:D_SOD-123, F.Cu at (247.3, -206.6)
- added D169: 1N4148W, Diode_SMD:D_SOD-123, F.Cu at (314.0, -172.8)
- added D17: SK6812, LED_SMD:LED_SK6812_PLCC4_5.0x5.0mm_P3.2mm, F.Cu at (9.53, -376.6)
- added D170: 1N4148W, Diode_SMD:D_SOD-123, F.Cu at (293.8, -152.3)
- added D171: 1N4148W, Diode_SMD:D_SOD-123, F.Cu at (182.9, -208.9)
- added D172: 1N4148W, Diode_SMD:D_SOD-123, F.Cu at (310.9, -179.6)
- added D173: 1N4148W, Diode_SMD:D_SOD-123, F.Cu at (302.5, -172.3)
- added D174: 1N4148W, Diode_SMD:D_SOD-123, F.Cu at (282.3, -152.1)
- added D175: 1N4148W, Diode_SMD:D_SOD-123, F.Cu at (191.9, -191.6)
- added D176: 1N4148W, Diode_SMD:D_SOD-123, F.Cu at (331.1, -199.5)
- added D177: SK6812, LED_SMD:LED_SK6812_PLCC4_5.0x5.0mm_P3.2mm, F.Cu at (216.8, -233.4)
- added D178: SK6812, LED_SMD:LED_SK6812_PLCC4_5.0x5.0mm_P3.2mm, F.Cu at (283.6, -163.7)
- added D179: SK6812, LED_SMD:LED_SK6812_PLCC4_5.0x5.0mm_P3.2mm, F.Cu at (303.8, -183.9)
- added D18: SK6812, LED_SMD:LED_SK6812_PLCC4_5.0x5.0mm_P3.2mm, F.Cu at (28.4, -376.6)
- added D180: SK6812, LED_SMD:LED_SK6812_PLCC4_5.0x5.0mm_P3.2mm, F.Cu at (295.4, -177.3)
- added D181: SK6812, LED_SMD:LED_SK6812_PLCC4_5.0x5.0mm_P3.2mm, F.Cu at (332.4, -211.1)
- added D182: SK6812, LED_SMD:LED_SK6812_PLCC4_5.0x5.0mm_P3.2mm, F.Cu at (177.8, -220.6)
- added D183: SK6812, LED_SMD:LED_SK6812_PLCC4_5.0x5.0mm_P3.2mm, F.Cu at (340.9, -218.0)
- added D184: SK6812, LED_SMD:LED_SK6812_PLCC4_5.0x5.0mm_P3.2mm, F.Cu at (155.9, -200.3)
- added D185: SK6812, LED_SMD:LED_SK6812_PLCC4_5.0x5.0mm_P3.2mm, F.Cu at (315.6, -191.2)
- added D186: SK6812, LED_SMD:LED_SK6812_PLCC4_5.0x5.0mm_P3.2mm, F.Cu at (186.2, -227.2)
- added D187: SK6812, LED_SMD:LED_SK6812_PLCC4_5.0x5.0mm_P3.2mm, F.Cu at (164.3, -207.0)
- added D188: SK6812, LED_SMD:LED_SK6812_PLCC4_5.0x5.0mm_P3.2mm, F.Cu at (188.2, -200.0)
- added D189: SK6812, LED_SMD:LED_SK6812_PLCC4_5.0x5.0mm_P3.2mm, F.Cu at (208.4, -220.2)
- added D19: SK6812, LED_SMD:LED_SK6812_PLCC4_5.0x5.0mm_P3.2mm, F.Cu at (47.5, -376.6)
- added D190: SK6812, LED_SMD:LED_SK6812_PLCC4_5.0x5.0mm_P3.2mm, F.Cu at (196.6, -206.6)
- added D191: SK6812, LED_SMD:LED_SK6812_PLCC4_5.0x5.0mm_P3.2mm, F.Cu at (228.6, -240.4)
- added D192: SK6812, LED_SMD:LED_SK6812_PLCC4_5.0x5.0mm_P3.2mm, F.Cu at (172.7, -213.6)
- added D193: 1N4148W, Diode_SMD:D_SOD-123, B.Cu at (124.8, -227.6)
- added D194: SK6812, LED_SMD:LED_SK6812_PLCC4_5.0x5.0mm_P3.2mm, F.Cu at (303.8, -177.3)
- added D2: 1N4148W, Diode_SMD:D_SOD-123, B.Cu at (36.8, -365.6)
- added D20: SK6812, LED_SMD:LED_SK6812_PLCC4_5.0x5.0mm_P3.2mm, F.Cu at (66.6, -376.6)
- added D21: SK6812, LED_SMD:LED_SK6812_PLCC4_5.0x5.0mm_P3.2mm, F.Cu at (85.7, -376.6)
- added D22: SK6812, LED_SMD:LED_SK6812_PLCC4_5.0x5.0mm_P3.2mm, F.Cu at (104.8, -376.6)
- added D23: SK6812, LED_SMD:LED_SK6812_PLCC4_5.0x5.0mm_P3.2mm, F.Cu at (123.8, -376.6)
- added D24: SK6812, LED_SMD:LED_SK6812_PLCC4_5.0x5.0mm_P3.2mm, F.Cu at (142.9, -376.6)
- added D25: SK6812, LED_SMD:LED_SK6812_PLCC4_5.0x5.0mm_P3.2mm, F.Cu at (161.9, -376.6)
- added D26: SK6812, LED_SMD:LED_SK6812_PLCC4_5.0x5.0mm_P3.2mm, F.Cu at (181.0, -376.6)
- added D27: SK6812, LED_SMD:LED_SK6812_PLCC4_5.0x5.0mm_P3.2mm, F.Cu at (200.0, -376.6)
- added D28: SK6812, LED_SMD:LED_SK6812_PLCC4_5.0x5.0mm_P3.2mm, F.Cu at (219.2, -376.6)
- added D29: SK6812, LED_SMD:LED_SK6812_PLCC4_5.0x5.0mm_P3.2mm, F.Cu at (238.1, -376.6)
- added D3: 1N4148W, Diode_SMD:D_SOD-123, B.Cu at (55.9, -365.6)
- added D30: SK6812, LED_SMD:LED_SK6812_PLCC4_5.0x5.0mm_P3.2mm, F.Cu at (257.3, -376.6)
- added D31: SK6812, LED_SMD:LED_SK6812_PLCC4_5.0x5.0mm_P3.2mm, F.Cu at (276.4, -376.6)
- added D32: SK6812, LED_SMD:LED_SK6812_PLCC4_5.0x5.0mm_P3.2mm, F.Cu at (80.1, -200.3)
- added D33: 1N4148W, Diode_SMD:D_SOD-123, B.Cu at (17.8, -346.5)
- added D34: 1N4148W, Diode_SMD:D_SOD-123, B.Cu at (36.8, -346.5)
- added D35: 1N4148W, Diode_SMD:D_SOD-123, B.Cu at (55.9, -346.5)
- added D36: 1N4148W, Diode_SMD:D_SOD-123, B.Cu at (74.9, -346.5)
- added D37: 1N4148W, Diode_SMD:D_SOD-123, B.Cu at (94.0, -346.5)
- added D38: 1N4148W, Diode_SMD:D_SOD-123, B.Cu at (113.0, -346.5)
- added D39: 1N4148W, Diode_SMD:D_SOD-123, B.Cu at (132.1, -346.5)
- added D4: 1N4148W, Diode_SMD:D_SOD-123, B.Cu at (74.9, -365.6)
- added D40: 1N4148W, Diode_SMD:D_SOD-123, B.Cu at (151.3, -346.5)
- added D41: 1N4148W, Diode_SMD:D_SOD-123, B.Cu at (170.2, -346.5)
- added D42: 1N4148W, Diode_SMD:D_SOD-123, B.Cu at (189.2, -346.5)
- added D43: 1N4148W, Diode_SMD:D_SOD-123, B.Cu at (208.3, -346.5)
- added D44: 1N4148W, Diode_SMD:D_SOD-123, B.Cu at (227.3, -346.5)
- added D45: 1N4148W, Diode_SMD:D_SOD-123, B.Cu at (246.4, -346.5)
- added D46: 1N4148W, Diode_SMD:D_SOD-123, B.Cu at (275.0, -346.5)
- added D47: 1N4148W, Diode_SMD:D_SOD-123, B.Cu at (303.5, -346.5)
- added D48: 1N4148W, Diode_SMD:D_SOD-123, B.Cu at (322.6, -346.5)
- added D49: SK6812, LED_SMD:LED_SK6812_PLCC4_5.0x5.0mm_P3.2mm, F.Cu at (9.53, -357.5)
- added D5: 1N4148W, Diode_SMD:D_SOD-123, B.Cu at (94.0, -365.6)
- added D50: SK6812, LED_SMD:LED_SK6812_PLCC4_5.0x5.0mm_P3.2mm, F.Cu at (28.4, -357.5)
- added D51: SK6812, LED_SMD:LED_SK6812_PLCC4_5.0x5.0mm_P3.2mm, F.Cu at (47.5, -357.5)
- added D52: SK6812, LED_SMD:LED_SK6812_PLCC4_5.0x5.0mm_P3.2mm, F.Cu at (66.5, -357.5)
- added D53: SK6812, LED_SMD:LED_SK6812_PLCC4_5.0x5.0mm_P3.2mm, F.Cu at (85.7, -357.5)
- added D54: SK6812, LED_SMD:LED_SK6812_PLCC4_5.0x5.0mm_P3.2mm, F.Cu at (104.7, -357.6)
- added D55: SK6812, LED_SMD:LED_SK6812_PLCC4_5.0x5.0mm_P3.2mm, F.Cu at (123.8, -357.5)
- added D56: SK6812, LED_SMD:LED_SK6812_PLCC4_5.0x5.0mm_P3.2mm, F.Cu at (142.9, -357.5)
- added D57: SK6812, LED_SMD:LED_SK6812_PLCC4_5.0x5.0mm_P3.2mm, F.Cu at (161.9, -357.5)
- added D58: SK6812, LED_SMD:LED_SK6812_PLCC4_5.0x5.0mm_P3.2mm, F.Cu at (181.0, -357.5)
- added D59: SK6812, LED_SMD:LED_SK6812_PLCC4_5.0x5.0mm_P3.2mm, F.Cu at (200.0, -357.5)
- added D6: 1N4148W, Diode_SMD:D_SOD-123, B.Cu at (113.0, -365.6)
- added D60: SK6812, LED_SMD:LED_SK6812_PLCC4_5.0x5.0mm_P3.2mm, F.Cu at (219.2, -357.5)
- added D61: SK6812, LED_SMD:LED_SK6812_PLCC4_5.0x5.0mm_P3.2mm, F.Cu at (238.1, -357.5)
- added D62: SK6812, LED_SMD:LED_SK6812_PLCC4_5.0x5.0mm_P3.2mm, F.Cu at (266.7, -357.5)
- added D63: SK6812, LED_SMD:LED_SK6812_PLCC4_5.0x5.0mm_P3.2mm, F.Cu at (295.3, -357.5)
- added D64: SK6812, LED_SMD:LED_SK6812_PLCC4_5.0x5.0mm_P3.2mm, F.Cu at (314.3, -357.5)
- added D65: 1N4148W, Diode_SMD:D_SOD-123, B.Cu at (341.5, -346.2)
- added D66: 1N4148W, Diode_SMD:D_SOD-123, B.Cu at (360.7, -346.2)
- added D67: 1N4148W, Diode_SMD:D_SOD-123, B.Cu at (22.5, -327.4)
- added D68: 1N4148W, Diode_SMD:D_SOD-123, B.Cu at (46.4, -327.4)
- added D69: 1N4148W, Diode_SMD:D_SOD-123, B.Cu at (65.4, -327.4)
- added D7: 1N4148W, Diode_SMD:D_SOD-123, B.Cu at (132.1, -365.6)
- added D70: 1N4148W, Diode_SMD:D_SOD-123, B.Cu at (84.5, -327.4)
- added D71: 1N4148W, Diode_SMD:D_SOD-123, B.Cu at (103.5, -327.4)
- added D72: 1N4148W, Diode_SMD:D_SOD-123, B.Cu at (122.6, -327.4)
- added D73: 1N4148W, Diode_SMD:D_SOD-123, B.Cu at (141.6, -327.4)
- added D74: 1N4148W, Diode_SMD:D_SOD-123, B.Cu at (160.7, -327.4)
- added D75: 1N4148W, Diode_SMD:D_SOD-123, B.Cu at (179.7, -327.4)
- added D76: 1N4148W, Diode_SMD:D_SOD-123, B.Cu at (198.8, -327.4)
- added D77: 1N4148W, Diode_SMD:D_SOD-123, B.Cu at (217.8, -327.4)
- added D78: 1N4148W, Diode_SMD:D_SOD-123, B.Cu at (236.9, -327.4)
- added D79: 1N4148W, Diode_SMD:D_SOD-123, B.Cu at (255.9, -327.4)
- added D8: 1N4148W, Diode_SMD:D_SOD-123, B.Cu at (151.1, -365.6)
- added D80: 1N4148W, Diode_SMD:D_SOD-123, B.Cu at (282.1, -317.9)
- added D81: SK6812, LED_SMD:LED_SK6812_PLCC4_5.0x5.0mm_P3.2mm, F.Cu at (333.4, -357.5)
- added D82: SK6812, LED_SMD:LED_SK6812_PLCC4_5.0x5.0mm_P3.2mm, F.Cu at (352.3, -357.5)
- added D83: SK6812, LED_SMD:LED_SK6812_PLCC4_5.0x5.0mm_P3.2mm, F.Cu at (14.2, -338.5)
- added D84: SK6812, LED_SMD:LED_SK6812_PLCC4_5.0x5.0mm_P3.2mm, F.Cu at (38.1, -338.5)
- added D85: SK6812, LED_SMD:LED_SK6812_PLCC4_5.0x5.0mm_P3.2mm, F.Cu at (57.1, -338.5)
- added D86: SK6812, LED_SMD:LED_SK6812_PLCC4_5.0x5.0mm_P3.2mm, F.Cu at (76.2, -338.5)
- added D87: SK6812, LED_SMD:LED_SK6812_PLCC4_5.0x5.0mm_P3.2mm, F.Cu at (95.1, -338.5)
- added D88: SK6812, LED_SMD:LED_SK6812_PLCC4_5.0x5.0mm_P3.2mm, F.Cu at (114.3, -338.5)
- added D89: SK6812, LED_SMD:LED_SK6812_PLCC4_5.0x5.0mm_P3.2mm, F.Cu at (133.3, -338.5)
- added D9: 1N4148W, Diode_SMD:D_SOD-123, B.Cu at (170.2, -365.6)
- added D90: SK6812, LED_SMD:LED_SK6812_PLCC4_5.0x5.0mm_P3.2mm, F.Cu at (152.4, -338.5)
- added D91: SK6812, LED_SMD:LED_SK6812_PLCC4_5.0x5.0mm_P3.2mm, F.Cu at (171.4, -338.5)
- added D92: SK6812, LED_SMD:LED_SK6812_PLCC4_5.0x5.0mm_P3.2mm, F.Cu at (190.5, -338.5)
- added D93: SK6812, LED_SMD:LED_SK6812_PLCC4_5.0x5.0mm_P3.2mm, F.Cu at (209.6, -338.5)
- added D94: SK6812, LED_SMD:LED_SK6812_PLCC4_5.0x5.0mm_P3.2mm, F.Cu at (228.6, -338.5)
- added D95: SK6812, LED_SMD:LED_SK6812_PLCC4_5.0x5.0mm_P3.2mm, F.Cu at (247.7, -338.5)
- added D96: SK6812, LED_SMD:LED_SK6812_PLCC4_5.0x5.0mm_P3.2mm, F.Cu at (273.9, -328.9)
- added D97: 1N4148W, Diode_SMD:D_SOD-123, B.Cu at (303.5, -327.3)
- added D98: 1N4148W, Diode_SMD:D_SOD-123, B.Cu at (322.6, -327.3)
- added D99: 1N4148W, Diode_SMD:D_SOD-123, B.Cu at (341.6, -327.3)
- added F1: 500mA, Fuse:Fuse_1206_3216Metric, F.Cu at (162.9, -198.7)
- added H1: MountingHole_Pad, MountingHole:MountingHole_2.2mm_M2_Pad_Via, F.Cu at (23.7, -230.8)
- added H2: MountingHole_Pad, MountingHole:MountingHole_2.2mm_M2_Pad_Via, F.Cu at (64.5, -247.0)
- added H3: MountingHole_Pad, MountingHole:MountingHole_2.2mm_M2_Pad_Via, F.Cu at (47.4, -240.0)
- added H4: MountingHole_Pad, MountingHole:MountingHole_2.2mm_M2_Pad_Via, F.Cu at (35.6, -236.6)
- added H5: MountingHole_Pad, MountingHole:MountingHole_2.2mm_M2_Pad_Via, F.Cu at (58.3, -244.5)
- added H6: MountingHole_Pad, MountingHole:MountingHole_2.2mm_M2_Pad_Via, F.Cu at (70.7, -237.6)
- added J1: USB_C_Receptacle_USB2.0, Connector_USB:USB_C_Receptacle_HRO_TYPE-C-31-M-12, F.Cu at (339.9, -377.7)
- added J2: ISP, Connector_PinHeader_2.54mm:PinHeader_2x03_P2.54mm_Vertical, F.Cu at (337.4, -364.6)
- added R1: 10k, Resistor_SMD:R_0805_2012Metric, F.Cu at (301.5, -159.1)
- added R2: 330, Resistor_SMD:R_0805_2012Metric, F.Cu at (234.7, -228.8)
- added R3: 22, Resistor_SMD:R_0805_2012Metric, F.Cu at (214.5, -208.6)
- added R4: 22, Resistor_SMD:R_0805_2012Metric, F.Cu at (220.6, -218.6)
- added R5: 10k, Resistor_SMD:R_0805_2012Metric, F.Cu at (208.5, -201.7)
- added R6: 22, Resistor_SMD:R_0805_2012Metric, F.Cu at (313.3, -169.7)
- added R7: 22, Resistor_SMD:R_0805_2012Metric, F.Cu at (349.0, -366.0)
- added SW1: SW_Push, Button_Switch_Keyboard:SW_Cherry_MX_1.00u_PCB, F.Cu at (6.99, -366.4)
- added SW10: SW_Push, Button_Switch_Keyboard:SW_Cherry_MX_1.00u_PCB, F.Cu at (178.4, -366.4)
- added SW11: SW_Push, Button_Switch_Keyboard:SW_Cherry_MX_1.00u_PCB, F.Cu at (197.5, -366.4)
- added SW12: SW_Push, Button_Switch_Keyboard:SW_Cherry_MX_1.00u_PCB, F.Cu at (216.5, -366.4)
- added SW13: SW_Push, Button_Switch_Keyboard:SW_Cherry_MX_1.00u_PCB, F.Cu at (235.6, -366.4)
- added SW14: SW_Push, Button_Switch_Keyboard:SW_Cherry_MX_1.00u_PCB, F.Cu at (254.6, -366.4)
- added SW15: SW_Push, Button_Switch_Keyboard:SW_Cherry_MX_1.00u_PCB, F.Cu at (273.7, -366.4)
- added SW16: SW_Push, Button_Switch_Keyboard:SW_Cherry_MX_1.00u_PCB, F.Cu at (330.8, -271.1)
- added SW18: SW_Push, Button_Switch_Keyboard:SW_Cherry_MX_1.00u_PCB, F.Cu at (6.99, -347.3)
- added SW19: SW_Push, Button_Switch_Keyboard:SW_Cherry_MX_1.00u_PCB, F.Cu at (26.0, -347.3)
- added SW2: SW_Push, Button_Switch_Keyboard:SW_Cherry_MX_1.00u_PCB, F.Cu at (26.0, -366.4)
- added SW20: SW_Push, Button_Switch_Keyboard:SW_Cherry_MX_1.00u_PCB, F.Cu at (45.1, -347.3)
- added SW21: SW_Push, Button_Switch_Keyboard:SW_Cherry_MX_1.00u_PCB, F.Cu at (64.1, -347.3)
- added SW22: SW_Push, Button_Switch_Keyboard:SW_Cherry_MX_1.00u_PCB, F.Cu at (83.2, -347.3)
- added SW23: SW_Push, Button_Switch_Keyboard:SW_Cherry_MX_1.00u_PCB, F.Cu at (102.2, -347.3)
- added SW24: SW_Push, Button_Switch_Keyboard:SW_Cherry_MX_1.00u_PCB, F.Cu at (121.3, -347.3)
- added SW25: SW_Push, Button_Switch_Keyboard:SW_Cherry_MX_1.00u_PCB, F.Cu at (140.3, -347.3)
- added SW26: SW_Push, Button_Switch_Keyboard:SW_Cherry_MX_1.00u_PCB, F.Cu at (159.4, -347.3)
- added SW27: SW_Push, Button_Switch_Keyboard:SW_Cherry_MX_1.00u_PCB, F.Cu at (178.4, -347.3)
- added SW28: SW_Push, Button_Switch_Keyboard:SW_Cherry_MX_1.00u_PCB, F.Cu at (197.5, -347.3)
- added SW29: SW_Push, Button_Switch_Keyboard:SW_Cherry_MX_1.00u_PCB, F.Cu at (216.5, -347.3)
- added SW3: SW_Push, Button_Switch_Keyboard:SW_Cherry_MX_1.00u_PCB, F.Cu at (45.1, -366.4)
- added SW30: SW_Push, Button_Switch_Keyboard:SW_Cherry_MX_1.00u_PCB, F.Cu at (235.6, -347.3)
- added SW31: SW_Push, Button_Switch_Keyboard:SW_Cherry_MX_2.00u_PCB, F.Cu at (264.2, -347.3)
- added SW32: SW_Push, Button_Switch_Keyboard:SW_Cherry_MX_1.00u_PCB, F.Cu at (292.7, -347.3)
- added SW33: SW_Push, Button_Switch_Keyboard:SW_Cherry_MX_1.00u_PCB, F.Cu at (311.8, -347.3)
- added SW34: SW_Push, Button_Switch_Keyboard:SW_Cherry_MX_1.00u_PCB, F.Cu at (330.8, -347.3)
- added SW35: SW_Push, Button_Switch_Keyboard:SW_Cherry_MX_1.00u_PCB, F.Cu at (349.9, -347.3)
- added SW36: SW_Push, Button_Switch_Keyboard:SW_Cherry_MX_1.50u_PCB, F.Cu at (11.7, -328.3)
- added SW37: SW_Push, Button_Switch_Keyboard:SW_Cherry_MX_1.00u_PCB, F.Cu at (35.6, -328.3)
- added SW38: SW_Push, Button_Switch_Keyboard:SW_Cherry_MX_1.00u_PCB, F.Cu at (54.6, -328.3)
- added SW39: SW_Push, Button_Switch_Keyboard:SW_Cherry_MX_1.00u_PCB, F.Cu at (73.7, -328.3)
- added SW4: SW_Push, Button_Switch_Keyboard:SW_Cherry_MX_1.00u_PCB, F.Cu at (64.1, -366.4)
- added SW40: SW_Push, Button_Switch_Keyboard:SW_Cherry_MX_1.00u_PCB, F.Cu at (92.7, -328.3)
- added SW41: SW_Push, Button_Switch_Keyboard:SW_Cherry_MX_1.00u_PCB, F.Cu at (111.8, -328.3)
- added SW42: SW_Push, Button_Switch_Keyboard:SW_Cherry_MX_1.00u_PCB, F.Cu at (130.8, -328.3)
- added SW43: SW_Push, Button_Switch_Keyboard:SW_Cherry_MX_1.00u_PCB, F.Cu at (149.9, -328.3)
- added SW44: SW_Push, Button_Switch_Keyboard:SW_Cherry_MX_1.00u_PCB, F.Cu at (168.9, -328.3)
- added SW45: SW_Push, Button_Switch_Keyboard:SW_Cherry_MX_1.00u_PCB, F.Cu at (188.0, -328.3)
- added SW46: SW_Push, Button_Switch_Keyboard:SW_Cherry_MX_1.00u_PCB, F.Cu at (207.0, -328.3)
- added SW47: SW_Push, Button_Switch_Keyboard:SW_Cherry_MX_1.00u_PCB, F.Cu at (226.1, -328.3)
- added SW48: SW_Push, Button_Switch_Keyboard:SW_Cherry_MX_1.00u_PCB, F.Cu at (245.1, -328.3)
- added SW49: SW_Push, Button_Switch_Keyboard:SW_Cherry_MX_ISOEnter_PCB, F.Cu at (271.3, -318.8)
- added SW5: SW_Push, Button_Switch_Keyboard:SW_Cherry_MX_1.00u_PCB, F.Cu at (83.2, -366.4)
- added SW50: SW_Push, Button_Switch_Keyboard:SW_Cherry_MX_1.00u_PCB, F.Cu at (292.7, -328.3)
- added SW51: SW_Push, Button_Switch_Keyboard:SW_Cherry_MX_1.00u_PCB, F.Cu at (311.8, -328.3)
- added SW52: SW_Push, Button_Switch_Keyboard:SW_Cherry_MX_1.00u_PCB, F.Cu at (330.8, -328.3)
- added SW53: SW_Push, Button_Switch_Keyboard:SW_Cherry_MX_2.00u_Vertical_PCB, F.Cu at (349.9, -318.8)
- added SW54: SW_Push, Button_Switch_Keyboard:SW_Cherry_MX_1.75u_PCB, F.Cu at (14.1, -309.2)
- added SW55: SW_Push, Button_Switch_Keyboard:SW_Cherry_MX_1.00u_PCB, F.Cu at (40.4, -309.2)
- added SW56: SW_Push, Button_Switch_Keyboard:SW_Cherry_MX_1.00u_PCB, F.Cu at (59.4, -309.2)
- added SW57: SW_Push, Button_Switch_Keyboard:SW_Cherry_MX_1.00u_PCB, F.Cu at (78.5, -309.2)
- added SW58: SW_Push, Button_Switch_Keyboard:SW_Cherry_MX_1.00u_PCB, F.Cu at (97.5, -309.2)
- added SW59: SW_Push, Button_Switch_Keyboard:SW_Cherry_MX_1.00u_PCB, F.Cu at (116.6, -309.2)
- added SW6: SW_Push, Button_Switch_Keyboard:SW_Cherry_MX_1.00u_PCB, F.Cu at (102.2, -366.4)
- added SW60: SW_Push, Button_Switch_Keyboard:SW_Cherry_MX_1.00u_PCB, F.Cu at (135.6, -309.2)
- added SW61: SW_Push, Button_Switch_Keyboard:SW_Cherry_MX_1.00u_PCB, F.Cu at (154.7, -309.2)
- added SW62: SW_Push, Button_Switch_Keyboard:SW_Cherry_MX_1.00u_PCB, F.Cu at (173.7, -309.2)
- added SW63: SW_Push, Button_Switch_Keyboard:SW_Cherry_MX_1.00u_PCB, F.Cu at (192.8, -309.2)
- added SW64: SW_Push, Button_Switch_Keyboard:SW_Cherry_MX_1.00u_PCB, F.Cu at (211.8, -309.2)
- added SW65: SW_Push, Button_Switch_Keyboard:SW_Cherry_MX_1.00u_PCB, F.Cu at (230.9, -309.2)
- added SW66: SW_Push, Button_Switch_Keyboard:SW_Cherry_MX_1.00u_PCB, F.Cu at (249.9, -309.2)
- added SW67: SW_Push, Button_Switch_Keyboard:SW_Cherry_MX_1.00u_PCB, F.Cu at (292.7, -309.2)
- added SW68: SW_Push, Button_Switch_Keyboard:SW_Cherry_MX_1.00u_PCB, F.Cu at (311.8, -309.2)
- added SW69: SW_Push, Button_Switch_Keyboard:SW_Cherry_MX_1.00u_PCB, F.Cu at (330.8, -309.2)
- added SW7: SW_Push, Button_Switch_Keyboard:SW_Cherry_MX_1.00u_PCB, F.Cu at (121.3, -366.4)
- added SW70: SW_Push, Button_Switch_Keyboard:SW_Cherry_MX_2.00u_PCB, F.Cu at (16.5, -290.2)
- added SW71: SW_Push, Button_Switch_Keyboard:SW_Cherry_MX_1.00u_PCB, F.Cu at (45.1, -290.2)
- added SW72: SW_Push, Button_Switch_Keyboard:SW_Cherry_MX_1.00u_PCB, F.Cu at (64.1, -290.2)
- added SW73: SW_Push, Button_Switch_Keyboard:SW_Cherry_MX_1.00u_PCB, F.Cu at (83.2, -290.2)
- added SW74: SW_Push, Button_Switch_Keyboard:SW_Cherry_MX_1.00u_PCB, F.Cu at (102.2, -290.2)
- added SW75: SW_Push, Button_Switch_Keyboard:SW_Cherry_MX_1.00u_PCB, F.Cu at (121.3, -290.2)
- added SW76: SW_Push, Button_Switch_Keyboard:SW_Cherry_MX_1.00u_PCB, F.Cu at (140.3, -290.2)
- added SW77: SW_Push, Button_Switch_Keyboard:SW_Cherry_MX_1.00u_PCB, F.Cu at (159.4, -290.2)
- added SW78: SW_Push, Button_Switch_Keyboard:SW_Cherry_MX_1.00u_PCB, F.Cu at (178.4, -290.2)
- added SW79: SW_Push, Button_Switch_Keyboard:SW_Cherry_MX_1.00u_PCB, F.Cu at (197.5, -290.2)
- added SW8: SW_Push, Button_Switch_Keyboard:SW_Cherry_MX_1.00u_PCB, F.Cu at (140.3, -366.4)
- added SW80: SW_Push, Button_Switch_Keyboard:SW_Cherry_MX_1.00u_PCB, F.Cu at (216.5, -290.2)
- added SW81: SW_Push, Button_Switch_Keyboard:SW_Cherry_MX_1.00u_PCB, F.Cu at (235.6, -290.2)
- added SW82: SW_Push, Button_Switch_Keyboard:SW_Cherry_MX_1.00u_PCB, F.Cu at (254.6, -290.2)
- added SW83: SW_Push, Button_Switch_Keyboard:SW_Cherry_MX_1.00u_PCB, F.Cu at (273.7, -290.2)
- added SW84: SW_Push, Button_Switch_Keyboard:SW_Cherry_MX_1.00u_PCB, F.Cu at (292.7, -290.2)
- added SW85: SW_Push, Button_Switch_Keyboard:SW_Cherry_MX_1.00u_PCB, F.Cu at (311.8, -290.2)
- added SW86: SW_Push, Button_Switch_Keyboard:SW_Cherry_MX_1.00u_PCB, F.Cu at (330.8, -290.2)
- added SW87: SW_Push, Button_Switch_Keyboard:SW_Cherry_MX_2.00u_Vertical_PCB, F.Cu at (349.9, -280.7)
- added SW88: SW_Push, Button_Switch_Keyboard:SW_Cherry_MX_1.00u_PCB, F.Cu at (11.6, -271.1)
- added SW89: SW_Push, Button_Switch_Keyboard:SW_Cherry_MX_1.00u_PCB, F.Cu at (35.4, -271.1)
- added SW9: SW_Push, Button_Switch_Keyboard:SW_Cherry_MX_1.00u_PCB, F.Cu at (159.4, -366.4)
- added SW90: SW_Push, Button_Switch_Keyboard:SW_Cherry_MX_1.00u_PCB, F.Cu at (54.5, -271.1)
- added SW91: SW_Push, Button_Switch_Keyboard:SW_Cherry_MX_6.25u_PCB, F.Cu at (123.6, -271.1)
- added SW92: SW_Push, Button_Switch_Keyboard:SW_Cherry_MX_1.00u_PCB, F.Cu at (192.7, -271.1)
- added SW93: SW_Push, Button_Switch_Keyboard:SW_Cherry_MX_1.00u_PCB, F.Cu at (211.7, -271.1)
- added SW94: SW_Push, Button_Switch_Keyboard:SW_Cherry_MX_1.00u_PCB, F.Cu at (233.2, -271.1)
- added SW95: SW_Push, Button_Switch_Keyboard:SW_Cherry_MX_1.00u_PCB, F.Cu at (254.6, -271.1)
- added SW96: SW_Push, Button_Switch_Keyboard:SW_Cherry_MX_1.00u_PCB, F.Cu at (273.7, -271.1)
- added SW97: SW_Push, Button_Switch_Keyboard:SW_Cherry_MX_1.00u_PCB, F.Cu at (292.7, -271.1)
- added SW98: SW_Push, Button_Switch_Keyboard:SW_Cherry_MX_1.00u_PCB, F.Cu at (311.8, -271.1)
- added U1: CD74HC4067M, Package_SO:SOIC-24W_7.5x15.4mm_P1.27mm, F.Cu at (295.1, -372.0)
- added U2: ATmega32U4-AU, Package_QFP:TQFP-44_10x10mm_P0.8mm, F.Cu at (316.1, -372.0)
- added Y1: 16MHz, Crystal:Crystal_SMD_HC49-SD, F.Cu at (329.1, -372.1)

Commit message: working on pcb
Parts:
- C1, C2, C3, C4, C5, C6, C7, C8, D101, D102, D103, D104, D105, D106, D107, D108, D109, D110, D111, D112, D129, D130, D131, D132, D133, D134, D135, D136, D137, D138, D139, D140, D141, D142, D143, D144, D16, D161, D162, D163, D164, D165, D166, D167, D168, D169, D170, D171, D172, D173, D174, D175, D176: moved to B.Cu
- SW88: footprint Button_Switch_Keyboard:SW_Cherry_MX_1.00u_PCB -> Button_Switch_Keyboard:SW_Cherry_MX_1.50u_PCB
- SW94: footprint Button_Switch_Keyboard:SW_Cherry_MX_1.00u_PCB -> Button_Switch_Keyboard:SW_Cherry_MX_1.25u_PCB
- moved H5 540.3 mm to (380.0, 189.6)
- moved R7 533.1 mm to (393.8, 165.2)
- moved D183 524.5 mm to (41.9, 213.0)
- moved D193 504.6 mm to (350.3, 223.9)
- moved D167 504.3 mm to (50.2, 223.9), turned to 90 degrees
- moved C7 500.1 mm to (378.6, 124.5)
- moved D32 499.8 mm to (361.1, 213.0)
- moved U2 496.5 mm to (349.8, 123.4)
- moved C5 496.0 mm to (391.0, 124.5)
- moved SW88 495.1 mm to (39.4, 223.1)
- moved D1 495.1 mm to (45.5, 128.7)
- moved D10 495.1 mm to (216.9, 128.7)
- moved D100 495.1 mm to (388.4, 176.7)
- moved D11 495.1 mm to (236.0, 128.7)
- moved D113 495.1 mm to (323.0, 155.8)
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Connections:
- D16 pad 1: R0 -> R6
- D194 pad 4: (no net) -> Net-(D194-Pad4)
- D31 pad 4: Net-(D31-Pad4) -> LED1
- D32 pad 2: Net-(D31-Pad4) -> Net-(D194-Pad4)
- D32 pad 4: LED1 -> (no net)
- SW16 pad 1: C15 -> C1
Routing:
- net GND: track 0.00 -> 2360.6 mm, vias 0 -> 8
- net +5V: track 0.00 -> 2247.6 mm, vias 0 -> 3
- net C0: track 0.00 -> 530.2 mm, vias 0 -> 4
- net R5: track 0.00 -> 523.2 mm, vias 0 -> 1
- net C1: track 0.00 -> 522.4 mm, vias 0 -> 3
- net R3: track 0.00 -> 497.4 mm, vias 0 -> 7
- net C5: track 0.00 -> 463.8 mm, vias 0 -> 5
- net R4: track 0.00 -> 456.5 mm, vias 0 -> 7
- net C4: track 0.00 -> 453.9 mm, vias 0 -> 1
- net C2: track 0.00 -> 446.5 mm, vias 0 -> 2
- net C3: track 0.00 -> 432.1 mm, vias 0 -> 2
- net R1: track 0.00 -> 425.4 mm, vias 0 -> 3
- net R2: track 0.00 -> 392.7 mm, vias 0 -> 8
- net R0: track 0.00 -> 369.0 mm, vias 0 -> 1
- net Net-(D17-Pad2): track 0.00 -> 365.3 mm, vias 0 -> 2
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Other:
- board outline added: 375 x 125.6 mm
- board text added: "RCK v1.0 Jan. 2023"
- board text added: "Raúl Reinosa"

Commit message: continue working on pcb
Parts:
- J1: moved to B.Cu
- moved R2 354.3 mm to (40.6, 110.4), turned to 180 degrees
- moved C6 39.0 mm to (348.4, 112.2)
- moved R7 31.2 mm to (393.8, 134.0)
- moved C7 29.4 mm to (351.9, 112.2)
- moved C8 19.7 mm to (360.0, 124.3)
- moved J2 17.9 mm to (366.0, 117.6), turned to 180 degrees
- moved J1 12.9 mm to (377.0, 110.1), turned to 0 degrees
- moved R6 11.9 mm to (393.8, 148.5)
- moved R1 8.89 mm to (393.8, 143.5)
- moved C1 6.94 mm to (381.1, 125.2)
- moved R3 6.10 mm to (393.8, 138.7)
- moved R4 4.22 mm to (393.8, 154.4)
- moved R5 4.02 mm to (393.8, 159.3)
- moved F1 3.99 mm to (356.0, 112.0), turned to 90 degrees
- moved C3 2.37 mm to (384.7, 125.2)
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Connections:
- C5 pad 1: GND -> +5V
- C5 pad 2: +5V -> GND
- C8 pad 1: Net-(C8-Pad1) -> GND
- C8 pad 2: GND -> Net-(C8-Pad2)
- U2 pad 6: Net-(C8-Pad1) -> Net-(C8-Pad2)
Routing:
- net GND: track 2360.6 -> 0.00 mm, vias 8 -> 0
- net +5V: track 2247.6 -> 0.00 mm, vias 3 -> 0
- net C0: track 530.2 -> 0.00 mm, vias 4 -> 0
- net R5: track 523.2 -> 0.00 mm, vias 1 -> 0
- net C1: track 522.4 -> 0.00 mm, vias 3 -> 0
- net R3: track 497.4 -> 0.00 mm, vias 7 -> 0
- net C5: track 463.8 -> 0.00 mm, vias 5 -> 0
- net R4: track 456.5 -> 0.00 mm, vias 7 -> 0
- net C4: track 453.9 -> 0.00 mm, vias 1 -> 0
- net C2: track 446.5 -> 0.00 mm, vias 2 -> 0
- net C3: track 432.1 -> 0.00 mm, vias 2 -> 0
- net R1: track 425.4 -> 0.00 mm, vias 3 -> 0
- net R2: track 392.7 -> 0.00 mm, vias 8 -> 0
- net R0: track 369.0 -> 0.00 mm, vias 1 -> 0
- net Net-(D17-Pad2): track 365.3 -> 0.00 mm, vias 2 -> 0
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
Commit message: continue with pcb
Parts:
- removed D17: SK6812, LED_SMD:LED_SK6812_PLCC4_5.0x5.0mm_P3.2mm
- added H7: MountingHole_Pad, MountingHole:MountingHole_2.2mm_M2_Pad_Via, F.Cu at (26.7, 124.9)
- added H8: MountingHole_Pad, MountingHole:MountingHole_2.2mm_M2_Pad_Via, F.Cu at (26.7, 239.1)
- added H9: MountingHole_Pad, MountingHole:MountingHole_2.2mm_M2_Pad_Via, F.Cu at (388.6, 239.2)
- added L17: SK6812, LED_SMD:LED_SK6812_PLCC4_5.0x5.0mm_P3.2mm, F.Cu at (36.3, 129.4)
- moved H4 99.5 mm to (388.6, 144.1)
- moved R1 19.6 mm to (392.2, 163.0)
- moved R4 19.6 mm to (392.2, 173.8)
- moved R7 19.6 mm to (392.2, 153.5)
- moved R3 19.6 mm to (392.2, 158.2)
- moved R6 19.6 mm to (392.2, 168.0)
- moved R5 19.6 mm to (392.2, 178.8)
- moved C4 17.5 mm to (391.3, 137.7)
- moved F1 14.6 mm to (365.6, 122.9), turned to 0 degrees
- moved J2 14.4 mm to (366.5, 132.0)
- moved C1 13.5 mm to (376.2, 137.7)
- moved C2 13.5 mm to (383.6, 137.7)
- moved C3 13.5 mm to (379.9, 137.7)
- moved C5 13.5 mm to (387.4, 137.7)
- moved D193 11.7 mm to (349.3, 235.6)
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Other:
- outline, holes or cut-outs redrawn

Commit message: maybe first version
Parts:
- renumbered L17 to D17
Routing:
- net GND: track 0.00 -> 2416.5 mm, vias 0 -> 6
- net +5V: track 0.00 -> 2224.8 mm, vias 0 -> 1
- net C1: track 0.00 -> 541.3 mm, vias 0 -> 2
- net C2: track 0.00 -> 518.2 mm, vias 0 -> 1
- net C0: track 0.00 -> 513.0 mm, vias 0 -> 3
- net R3: track 0.00 -> 507.0 mm, vias 0 -> 7
- net R4: track 0.00 -> 506.1 mm, vias 0 -> 6
- net R5: track 0.00 -> 500.8 mm, vias 0 -> 1
- net R1: track 0.00 -> 480.1 mm, vias 0 -> 6
- net C5: track 0.00 -> 472.8 mm, vias 0 -> 2
- net C3: track 0.00 -> 469.8 mm, vias 0 -> 1
- net C4: track 0.00 -> 466.2 mm, vias 0 -> 2
- net R2: track 0.00 -> 407.9 mm, vias 0 -> 5
- net C6: track 0.00 -> 394.0 mm, vias 0 -> 1
- net R0: track 0.00 -> 355.3 mm, vias 0 -> 1
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
Commit message: still working on it
Parts:
- added C9: 100nF, Capacitor_SMD:C_0805_2012Metric, B.Cu at (372.5, 137.7)
Connections:
- U2 pad 42: (no net) -> Net-(C9-Pad1)
Routing:
- net Net-(C9-Pad1): track 0.00 -> 43.3 mm, vias 0 -> 3
- net GND: track 2416.5 -> 2434.2 mm
- net +5V: track 2224.8 -> 2228.7 mm
- net Net-(R5-Pad2): track 71.7 -> 75.3 mm
- net Net-(R3-Pad1): track 57.1 -> 58.5 mm
- net Net-(R4-Pad1): track 72.9 -> 74.1 mm
- net Net-(C7-Pad2): track 29.0 -> 29.8 mm
- net Net-(J1-PadA6): track 41.1 -> 41.7 mm
Other:
- rule trace_min: 0.2 -> 0.15
- rule via_min_size: 0.4 -> 0.3
