File: pcb/pcb.kicad_pcb (KiCad board)
At the start: 2 copper layers, 375 x 125.6 mm, 322 parts, among them J1 USB_C_Receptacle_USB2.0, J2 ISP, SW1 SW_Push, SW10 SW_Push, SW11 SW_Push, SW12 SW_Push, SW13 SW_Push, SW14 SW_Push, SW15 SW_Push, SW16 SW_Push, SW18 SW_Push, SW19 SW_Push, SW2 SW_Push, SW20 SW_Push, SW21 SW_Push, SW22 SW_Push, SW23 SW_Push, SW24 SW_Push, SW25 SW_Push, SW26 SW_Push, SW27 SW_Push, SW28 SW_Push, SW29 SW_Push, SW3 SW_Push, SW30 SW_Push, SW31 SW_Push, SW32 SW_Push, SW33 SW_Push, SW34 SW_Push, SW35 SW_Push, SW36 SW_Push, SW37 SW_Push, SW38 SW_Push, SW39 SW_Push, SW4 SW_Push, SW40 SW_Push, SW41 SW_Push, SW42 SW_Push, SW43 SW_Push, SW44 SW_Push, SW45 SW_Push, SW46 SW_Push, SW47 SW_Push, SW48 SW_Push, SW49 SW_Push, SW5 SW_Push, SW50 SW_Push, SW51 SW_Push, SW52 SW_Push, SW53 SW_Push, SW54 SW_Push, SW55 SW_Push, SW56 SW_Push, SW57 SW_Push, SW58 SW_Push, SW59 SW_Push, SW6 SW_Push, SW60 SW_Push, SW61 SW_Push, SW62 SW_Push, SW63 SW_Push, SW64 SW_Push, SW65 SW_Push, SW66 SW_Push, SW67 SW_Push, SW68 SW_Push, SW69 SW_Push, SW7 SW_Push, SW70 SW_Push, SW71 SW_Push, SW72 SW_Push, SW73 SW_Push, SW74 SW_Push, SW75 SW_Push, SW76 SW_Push, SW77 SW_Push, SW78 SW_Push, SW79 SW_Push, SW8 SW_Push, SW80 SW_Push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

Commit message: near to finish pcb
Parts:
- added H10: MountingHole_Pad, MountingHole:MountingHole_2.2mm_M2_Pad_Via, F.Cu at (174.4, 183.6)
- SW1, SW10, SW11, SW12, SW13, SW14, SW15, SW16, SW18, SW19, SW2, SW20, SW21, SW22, SW23, SW24, SW25, SW26, SW27, SW28, SW29, SW3, SW30, SW32, SW33, SW34, SW35, SW37, SW38, SW39, SW4, SW40, SW41, SW42, SW43, SW44, SW45, SW46, SW47, SW48, SW5, SW50, SW51, SW52, SW55, SW56, SW57, SW58, SW59, SW6, SW60, SW61, SW62, SW63, SW64, SW65, SW66, SW67, SW68, SW69, SW7, SW71, SW72, SW73, SW74, SW75, SW76, SW77, SW78, SW79, SW8, SW80, SW81, SW82, SW83, SW84, SW85, SW86, SW89, SW9, SW90, SW92, SW93, SW95, SW96, SW97, SW98: footprint Button_Switch_Keyboard:SW_Cherry_MX_1.00u_PCB -> Button_Switch_Keyboard:SW_Cherry_MX_1.00u_Plate
- SW36, SW88: footprint Button_Switch_Keyboard:SW_Cherry_MX_1.50u_PCB -> Button_Switch_Keyboard:SW_Cherry_MX_1.50u_Plate
- SW54: footprint Button_Switch_Keyboard:SW_Cherry_MX_1.75u_PCB -> Button_Switch_Keyboard:SW_Cherry_MX_1.00u_Plate
- SW94: footprint Button_Switch_Keyboard:SW_Cherry_MX_1.25u_PCB -> Button_Switch_Keyboard:SW_Cherry_MX_1.25u_Plate
- moved H2 315.4 mm to (379.0, 204.5)
- moved H4 260.3 mm to (141.7, 226.3)
- moved H1 252.2 mm to (307.1, 153.0)
- moved H5 171.2 mm to (217.2, 145.7)
- moved H9 114.0 mm to (289.6, 182.8)
- moved H6 86.2 mm to (379.2, 167.4)
- moved H3 78.8 mm to (141.0, 145.7)
- moved H8 44.9 mm to (61.3, 210.5)
- moved H7 28.2 mm to (45.8, 145.7)
Routing:
- net GND: track 2434.2 -> 0.00 mm, vias 6 -> 0
- net +5V: track 2228.7 -> 0.00 mm, vias 1 -> 0
- net C1: track 541.3 -> 0.00 mm, vias 2 -> 0
- net C2: track 518.2 -> 0.00 mm, vias 1 -> 0
- net C0: track 513.0 -> 0.00 mm, vias 3 -> 0
- net R3: track 507.0 -> 0.00 mm, vias 7 -> 0
- net R4: track 506.1 -> 0.00 mm, vias 6 -> 0
- net R5: track 500.8 -> 0.00 mm, vias 1 -> 0
- net R1: track 480.1 -> 0.00 mm, vias 6 -> 0
- net C5: track 472.8 -> 0.00 mm, vias 2 -> 0
- net C3: track 469.8 -> 0.00 mm, vias 1 -> 0
- net C4: track 466.2 -> 0.00 mm, vias 2 -> 0
- net R2: track 407.9 -> 0.00 mm, vias 5 -> 0
- net C6: track 394.0 -> 0.00 mm, vias 1 -> 0
- net R0: track 355.3 -> 0.00 mm, vias 1 -> 0
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
Commit message: near to have final version pcb ;)
Parts:
- SW54: footprint Button_Switch_Keyboard:SW_Cherry_MX_1.00u_Plate -> Button_Switch_Keyboard:SW_Cherry_MX_1.75u_Plate
Routing:
- net GND: track 0.00 -> 2400.6 mm, vias 0 -> 4
- net +5V: track 0.00 -> 2162.2 mm, vias 0 -> 2
- net C0: track 0.00 -> 540.2 mm, vias 0 -> 4
- net C1: track 0.00 -> 526.2 mm, vias 0 -> 5
- net R5: track 0.00 -> 494.3 mm, vias 0 -> 1
- net C5: track 0.00 -> 489.9 mm, vias 0 -> 3
- net R3: track 0.00 -> 486.3 mm, vias 0 -> 8
- net R2: track 0.00 -> 475.0 mm, vias 0 -> 3
- net C4: track 0.00 -> 468.9 mm, vias 0 -> 1
- net C2: track 0.00 -> 461.6 mm, vias 0 -> 2
- net C3: track 0.00 -> 435.0 mm, vias 0 -> 2
- net R4: track 0.00 -> 432.2 mm, vias 0 -> 7
- net R1: track 0.00 -> 409.0 mm, vias 0 -> 5
- net C6: track 0.00 -> 381.3 mm, vias 0 -> 1
- net R0: track 0.00 -> 367.4 mm, vias 0 -> 1
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
Commit message: continue working on pcb
Parts:
- moved R2 6.16 mm to (45.8, 122.4)
- moved D20 0.84 mm to (93.4, 128.5)
- moved D54 0.84 mm to (131.5, 147.6)
- moved D28 0.84 mm to (245.8, 128.6)
- moved D30 0.84 mm to (283.9, 128.6)
- moved D31 0.84 mm to (303.0, 128.6)
- moved D60 0.84 mm to (245.8, 147.6)
- moved D19 0.84 mm to (74.4, 128.6)
- moved D51 0.84 mm to (74.4, 147.6)
- moved D52 0.84 mm to (93.4, 147.6)
- moved D18 0.84 mm to (55.3, 128.6)
- moved D50 0.84 mm to (55.3, 147.6)
- moved D82 0.84 mm to (379.2, 147.6)
- moved D96 0.84 mm to (300.5, 176.2)
- moved D26 0.83 mm to (207.7, 128.6)
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Routing:
- net GND: track 2400.6 -> 0.00 mm, vias 4 -> 0
- net +5V: track 2162.2 -> 0.00 mm, vias 2 -> 0
- net C0: track 540.2 -> 0.00 mm, vias 4 -> 0
- net C1: track 526.2 -> 0.00 mm, vias 5 -> 0
- net R5: track 494.3 -> 0.00 mm, vias 1 -> 0
- net C5: track 489.9 -> 0.00 mm, vias 3 -> 0
- net R3: track 486.3 -> 0.00 mm, vias 8 -> 0
- net R2: track 475.0 -> 0.00 mm, vias 3 -> 0
- net C4: track 468.9 -> 0.00 mm, vias 1 -> 0
- net C2: track 461.6 -> 0.00 mm, vias 2 -> 0
- net C3: track 435.0 -> 0.00 mm, vias 2 -> 0
- net R4: track 432.2 -> 0.00 mm, vias 7 -> 0
- net R1: track 409.0 -> 0.00 mm, vias 5 -> 0
- net C6: track 381.3 -> 0.00 mm, vias 1 -> 0
- net R0: track 367.4 -> 0.00 mm, vias 1 -> 0
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Other:
- net class Default: trace_width 0.25 -> 0.15

Commit message: add test pcb
Parts:
- C1, C2, C3, C4, C5, C6, C7, C8, C9: footprint Capacitor_SMD:C_0805_2012Metric -> Capacitor_SMD:C_1206_3216Metric
- R1, R2, R3, R4, R5, R6, R7: footprint Resistor_SMD:R_0805_2012Metric -> Resistor_SMD:R_1206_3216Metric
- moved R7 7.43 mm to (392.2, 146.1)
- moved R3 6.73 mm to (392.2, 151.5)
- moved R1 6.10 mm to (392.2, 156.9)
- moved R4 5.64 mm to (392.3, 168.2)
- moved R6 5.60 mm to (392.3, 162.4)
- moved R5 5.16 mm to (392.3, 173.7)
- moved C6 4.20 mm to (351.7, 123.6)
- moved C7 4.20 mm to (355.2, 123.6)
- moved U2 3.86 mm to (346.0, 133.3)
- moved J2 3.82 mm to (367.9, 128.4), turned to 270 degrees
- moved U1 1.94 mm to (324.5, 133.5), turned to 90 degrees
- moved C8 1.58 mm to (359.2, 137.5)
- moved D150 0.83 mm to (74.4, 204.8)
- moved D191 0.83 mm to (303.0, 223.8)
- moved D118 0.83 mm to (69.7, 185.7)
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Other:
- board size 375 x 125.6 mm -> 375 x 125 mm

Commit message: maybe pcb done
Parts:
- moved H4 0.68 mm to (142.3, 226.0)
- moved H10 0.36 mm to (174.7, 183.9)
- moved H2 0.20 mm to (379.0, 204.3)
Routing:
- net +5V: track 0.00 -> 2203.4 mm, vias 0 -> 6
- net GND: track 0.00 -> 962.9 mm, vias 0 -> 5
- net R5: track 0.00 -> 533.0 mm, vias 0 -> 1
- net R1: track 0.00 -> 519.3 mm, vias 0 -> 3
- net C0: track 0.00 -> 518.9 mm, vias 0 -> 3
- net R3: track 0.00 -> 502.4 mm, vias 0 -> 8
- net C1: track 0.00 -> 492.2 mm, vias 0 -> 3
- net R2: track 0.00 -> 452.0 mm, vias 0 -> 6
- net C5: track 0.00 -> 444.6 mm, vias 0 -> 2
- net R4: track 0.00 -> 441.7 mm, vias 0 -> 7
- net C2: track 0.00 -> 438.3 mm, vias 0 -> 3
- net C4: track 0.00 -> 437.2 mm, vias 0 -> 1
- net C3: track 0.00 -> 420.1 mm, vias 0 -> 2
- net R0: track 0.00 -> 360.7 mm, vias 0 -> 1
- net C6: track 0.00 -> 354.8 mm, vias 0 -> 1
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- added copper zone on B.Cu, net GND
- added copper zone on F.Cu, net GND
Other:
- board text added: "Raúl Reinosa Simón"
- board text removed: "Raúl Reinosa"
