File: pcb/test/test.sch (KiCad schematic (older format))
At the start: 30 parts, among them J1 USB_C_Receptacle_USB2.0, J2 ISP, SW1 SW_Push, SW2 SW_Push, U1 ATmega32U4-AU, Y1 16MHz

Commit message: update budget
Parts:
- C7: value 100nF -> 0.1uF
Changed lines of the file:
@@
 P 1300 3250
 F 0 "C7" H 1392 3296 50  0000 L CNN
-F 1 "100nF" H 1392 3205 50  0000 L CNN
+F 1 "0.1uF" H 1392 3205 50  0000 L CNN
 F 2 "Capacitor_SMD:C_1206_3216Metric" H 1300 3250 50  0001 C CNN
 F 3 "~" H 1300 3250 50  0001 C CNN
