File: v1.0/plate/_autosave-plate.sch (KiCad schematic (older format))
At the start: 323 parts, among them J1 USB_C_Receptacle_USB2.0, J2 ISP, SW1 SW_Push, SW10 SW_Push, SW11 SW_Push, SW12 SW_Push, SW13 SW_Push, SW14 SW_Push, SW15 SW_Push, SW16 SW_Push, SW18 SW_Push, SW19 SW_Push, SW2 SW_Push, SW20 SW_Push, SW21 SW_Push, SW22 SW_Push, SW23 SW_Push, SW24 SW_Push, SW25 SW_Push, SW26 SW_Push, SW27 SW_Push, SW28 SW_Push, SW29 SW_Push, SW3 SW_Push, SW30 SW_Push, SW31 SW_Push, SW32 SW_Push, SW33 SW_Push, SW34 SW_Push, SW35 SW_Push, SW36 SW_Push, SW37 SW_Push, SW38 SW_Push, SW39 SW_Push, SW4 SW_Push, SW40 SW_Push, SW41 SW_Push, SW42 SW_Push, SW43 SW_Push, SW44 SW_Push, SW45 SW_Push, SW46 SW_Push, SW47 SW_Push, SW48 SW_Push, SW49 SW_Push, SW5 SW_Push, SW50 SW_Push, SW51 SW_Push, SW52 SW_Push, SW53 SW_Push, SW54 SW_Push, SW55 SW_Push, SW56 SW_Push, SW57 SW_Push, SW58 SW_Push, SW59 SW_Push, SW6 SW_Push, SW60 SW_Push, SW61 SW_Push, SW62 SW_Push, SW63 SW_Push, SW64 SW_Push, SW65 SW_Push, SW66 SW_Push, SW67 SW_Push, SW68 SW_Push, SW69 SW_Push, SW7 SW_Push, SW70 SW_Push, SW71 SW_Push, SW72 SW_Push, SW73 SW_Push, SW74 SW_Push, SW75 SW_Push, SW76 SW_Push, SW77 SW_Push, SW78 SW_Push, SW79 SW_Push, SW8 SW_Push, SW80 SW_Push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

Commit message: plate
Parts:
- removed C1, C2, C3, C5, C9: 0.1uF, Capacitor_SMD:C_1206_3216Metric, symbol Device:C_Small
- removed C4: 10uF, Capacitor_SMD:C_1206_3216Metric, symbol Device:C_Small
- removed C6, C7: 22uF, Capacitor_SMD:C_1206_3216Metric, symbol Device:C_Small
- removed C8: 1uF, Capacitor_SMD:C_1206_3216Metric, symbol Device:C_Small
- removed F1: 500mA, Fuse:Fuse_1206_3216Metric, symbol Device:Polyfuse
- removed J1: USB_C_Receptacle_USB2.0, Connector_USB:USB_C_Receptacle_HRO_TYPE-C-31-M-12, symbol Connector:USB_C_Receptacle_USB2.0
- removed J2: ISP, Connector_PinHeader_2.54mm:PinHeader_2x03_P2.54mm_Vertical, symbol Connector_Generic:Conn_02x03_Counter_Clockwise
- removed R1, R5: 10k, Resistor_SMD:R_1206_3216Metric, symbol Device:R_Small
- removed R3, R4, R6, R7: 22, Resistor_SMD:R_1206_3216Metric, symbol Device:R_Small
- removed U1: CD74HC4067M, Package_SO:SOIC-24W_7.5x15.4mm_P1.27mm, symbol 74xx:CD74HC4067M
- removed U2: ATmega32U4-AU, Package_QFP:TQFP-44_10x10mm_P0.8mm, symbol MCU_Microchip_ATmega:ATmega32U4-AU
- removed Y1: 16MHz, Crystal:Crystal_SMD_HC49-SD, symbol Device:Crystal_Small
- renumbered D102 to D100, D103 to D101, D104 to D102, D105 to D103, D106 to D104, D107 to D105, D108 to D106, D109 to D107, D110 to D108, D111 to D109, D112 to D110, D113 to D111, D114 to D112, D115 to D113, D116 to D114, D117 to D115, D118 to D116, D119 to D117, D120 to D118, D121 to D119, D122 to D120, D123 to D121, D124 to D122, D125 to D123, D126 to D124, D127 to D125, D128 to D126, D129 to D127, D130 to D128, D131 to D129, D132 to D130, D133 to D131, D134 to D132, D135 to D133, D136 to D134, D137 to D135, D138 to D136, D139 to D137, D140 to D138, D141 to D139, D142 to D140, D143 to D141, D144 to D142, D145 to D143, D146 to D144, D147 to D145, D148 to D146, D149 to D147, D150 to D148, D151 to D149, D152 to D150, D153 to D151, D154 to D152, D155 to D153, D156 to D154, D157 to D155, D158 to D156, D159 to D157, D160 to D158, D161 to D159, D17 to D16, D162 to D160, D163 to D161, D164 to D162, D165 to D163, D166 to D164, D167 to D165, D168 to D166, D169 to D167, D170 to D168, D171 to D169, D18 to D17, D172 to D170, D173 to D171, D174 to D172, D175 to D173, D176 to D174, D177 to D175, D178 to D176, D179 to D177, D180 to D178, D181 to D179, D19 to D18, D182 to D180, D183 to D181, D184 to D182, D185 to D183, D186 to D184, D187 to D185, D188 to D186, D189 to D187, D190 to D188, D191 to D189, D20 to D19, D192 to D190, D193 to D191, D16 to D192, D194 to D193, D32 to D194, D21 to D20, D22 to D21, D23 to D22, D24 to D23, D25 to D24, D26 to D25, D27 to D26, D28 to D27, D29 to D28, D30 to D29, D31 to D30, D33 to D31, D34 to D32, D35 to D33, D36 to D34, D37 to D35, D38 to D36, D39 to D37, D40 to D38, D41 to D39, D42 to D40, D43 to D41, D44 to D42, D45 to D43, D46 to D44, D47 to D45, D48 to D46, D49 to D47, D50 to D48, D51 to D49, D52 to D50, D53 to D51, D54 to D52, D55 to D53, D56 to D54, D57 to D55, D58 to D56, D59 to D57, D60 to D58, D61 to D59, D62 to D60, D63 to D61, D64 to D62, D65 to D63, D66 to D64, D67 to D65, D68 to D66, D69 to D67, D70 to D68, D71 to D69, D72 to D70, D73 to D71, D74 to D72, D75 to D73, D76 to D74, D77 to D75, D78 to D76, D79 to D77, D80 to D78, D81 to D79, D82 to D80, D83 to D81, D84 to D82, D85 to D83, D86 to D84, D87 to D85, D88 to D86, D89 to D87, D90 to D88, D91 to D89, D92 to D90, D93 to D91, D94 to D92, D95 to D93, D96 to D94, D97 to D95, D98 to D96, D99 to D97, D100 to D98, D101 to D99, R2 to R4, SW18 to SW16, SW19 to SW17, SW20 to SW18, SW21 to SW19, SW22 to SW20, SW23 to SW21, SW24 to SW22, SW25 to SW23, SW26 to SW24, SW27 to SW25, SW28 to SW26, SW29 to SW27, SW30 to SW28, SW31 to SW29, SW32 to SW30, SW33 to SW31, SW34 to SW32, SW35 to SW33, SW36 to SW34, SW37 to SW35, SW38 to SW36, SW39 to SW37, SW40 to SW38, SW41 to SW39, SW42 to SW40, SW43 to SW41, SW44 to SW42, SW45 to SW43, SW46 to SW44, SW47 to SW45, SW48 to SW46, SW49 to SW47, SW50 to SW48, SW51 to SW49, SW52 to SW50, SW53 to SW51, SW54 to SW52, SW55 to SW53, SW56 to SW54, SW57 to SW55, SW58 to SW56, SW59 to SW57, SW60 to SW58, SW61 to SW59, SW62 to SW60, SW63 to SW61, SW64 to SW62, SW65 to SW63, SW66 to SW64, SW67 to SW65, SW68 to SW66, SW69 to SW67, SW70 to SW68, SW71 to SW69, SW72 to SW70, SW73 to SW71, SW74 to SW72, SW75 to SW73, SW76 to SW74, SW77 to SW75, SW78 to SW76, SW79 to SW77, SW80 to SW78, SW81 to SW79, SW82 to SW80, SW83 to SW81, SW84 to SW82, SW85 to SW83, SW86 to SW84, SW87 to SW85, SW88 to SW86, SW89 to SW87, SW90 to SW88, SW91 to SW89, SW92 to SW90, SW93 to SW91, SW94 to SW92, SW95 to SW93, SW96 to SW94, SW97 to SW95, SW98 to SW96, SW16 to SW97
Connections:
- net labels removed: COM, D+, D-, MISO, MOSI, S0, S1, S2, S3, SCK, SE
- wire segments 686 -> 608
- no-connect marks 16 -> 3
