File: v1.0/plate/plate.kicad_pcb (KiCad board)
At the start: 2 copper layers, 375 x 125 mm, 107 parts, among them SW1 SW_Push, SW10 SW_Push, SW11 SW_Push, SW12 SW_Push, SW13 SW_Push, SW14 SW_Push, SW15 SW_Push, SW16 SW_Push, SW18 SW_Push, SW19 SW_Push, SW2 SW_Push, SW20 SW_Push, SW21 SW_Push, SW22 SW_Push, SW23 SW_Push, SW24 SW_Push, SW25 SW_Push, SW26 SW_Push, SW27 SW_Push, SW28 SW_Push, SW29 SW_Push, SW3 SW_Push, SW30 SW_Push, SW31 SW_Push, SW32 SW_Push, SW33 SW_Push, SW34 SW_Push, SW35 SW_Push, SW36 SW_Push, SW37 SW_Push, SW38 SW_Push, SW39 SW_Push, SW4 SW_Push, SW40 SW_Push, SW41 SW_Push, SW42 SW_Push, SW43 SW_Push, SW44 SW_Push, SW45 SW_Push, SW46 SW_Push, SW47 SW_Push, SW48 SW_Push, SW49 SW_Push, SW5 SW_Push, SW50 SW_Push, SW51 SW_Push, SW52 SW_Push, SW53 SW_Push, SW54 SW_Push, SW55 SW_Push, SW56 SW_Push, SW57 SW_Push, SW58 SW_Push, SW59 SW_Push, SW6 SW_Push, SW60 SW_Push, SW61 SW_Push, SW62 SW_Push, SW63 SW_Push, SW64 SW_Push, SW65 SW_Push, SW66 SW_Push, SW67 SW_Push, SW68 SW_Push, SW69 SW_Push, SW7 SW_Push, SW70 SW_Push, SW71 SW_Push, SW72 SW_Push, SW73 SW_Push, SW74 SW_Push, SW75 SW_Push, SW76 SW_Push, SW77 SW_Push, SW78 SW_Push, SW79 SW_Push, SW8 SW_Push, SW80 SW_Push, SW81 SW_Push, SW82 SW_Push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

Commit message: plate
Parts:
- removed H1, H10, H2, H3, H4, H5, H6, H7, H8, H9: MountingHole_Pad, MountingHole:MountingHole_2.2mm_M2_Pad_Via
- removed the SW70 at (43.2, 215.8)
- renumbered SW18 to SW16, SW19 to SW17, SW20 to SW18, SW21 to SW19, SW22 to SW20, SW23 to SW21, SW24 to SW22, SW25 to SW23, SW26 to SW24, SW27 to SW25, SW28 to SW26, SW29 to SW27, SW30 to SW28, SW31 to SW29, SW32 to SW30, SW33 to SW31, SW34 to SW32, SW35 to SW33, SW36 to SW34, SW37 to SW35, SW38 to SW36, SW39 to SW37, SW40 to SW38, SW41 to SW39, SW42 to SW40, SW43 to SW41, SW44 to SW42, SW45 to SW43, SW46 to SW44, SW47 to SW45, SW48 to SW46, SW49 to SW47, SW50 to SW48, SW51 to SW49, SW52 to SW50, SW53 to SW51, SW54 to SW52, SW55 to SW53, SW56 to SW54, SW57 to SW55, SW58 to SW56, SW59 to SW57, SW60 to SW58, SW61 to SW59, SW62 to SW60, SW63 to SW61, SW64 to SW62, SW65 to SW63, SW66 to SW64, SW67 to SW65, SW68 to SW66, SW69 to SW67, SW71 to SW69, SW72 to SW70, SW73 to SW71, SW74 to SW72, SW75 to SW73, SW76 to SW74, SW77 to SW75, SW78 to SW76, SW79 to SW77, SW80 to SW78, SW81 to SW79, SW82 to SW80, SW83 to SW81, SW84 to SW82, SW85 to SW83, SW86 to SW84, SW87 to SW85, SW88 to SW86, SW89 to SW87, SW90 to SW88, SW91 to SW89, SW92 to SW90, SW93 to SW91, SW94 to SW92, SW95 to SW93, SW96 to SW94, SW97 to SW95, SW98 to SW96, SW16 to SW97
Connections:
- SW1 pad 1: (no net) -> C0
- SW1 pad 2: (no net) -> Net-(D1-Pad2)
- SW10 pad 1: (no net) -> C9
- SW10 pad 2: (no net) -> Net-(D10-Pad2)
- SW11 pad 1: (no net) -> C10
- SW11 pad 2: (no net) -> Net-(D11-Pad2)
- SW12 pad 1: (no net) -> C11
- SW12 pad 2: (no net) -> Net-(D12-Pad2)
- SW13 pad 1: (no net) -> C12
- SW13 pad 2: (no net) -> Net-(D13-Pad2)
- SW14 pad 1: (no net) -> C13
- SW14 pad 2: (no net) -> Net-(D14-Pad2)
- SW15 pad 1: (no net) -> C14
- SW15 pad 2: (no net) -> Net-(D15-Pad2)
- SW16 pad 1: (no net) -> C0
- SW16 pad 2: (no net) -> Net-(D31-Pad2)
- SW17 pad 1: (no net) -> C1
- SW17 pad 2: (no net) -> Net-(D32-Pad2)
- SW18 pad 1: (no net) -> C2
- SW18 pad 2: (no net) -> Net-(D33-Pad2)
- SW19 pad 1: (no net) -> C3
- SW19 pad 2: (no net) -> Net-(D34-Pad2)
- SW2 pad 1: (no net) -> C1
- SW2 pad 2: (no net) -> Net-(D2-Pad2)
- SW20 pad 1: (no net) -> C4
- SW20 pad 2: (no net) -> Net-(D35-Pad2)
- SW21 pad 1: (no net) -> C5
- SW21 pad 2: (no net) -> Net-(D36-Pad2)
- SW22 pad 1: (no net) -> C6
- SW22 pad 2: (no net) -> Net-(D37-Pad2)
- SW23 pad 1: (no net) -> C7
- SW23 pad 2: (no net) -> Net-(D38-Pad2)
- SW24 pad 1: (no net) -> C8
- SW24 pad 2: (no net) -> Net-(D39-Pad2)
- SW25 pad 1: (no net) -> C9
- SW25 pad 2: (no net) -> Net-(D40-Pad2)
- SW26 pad 1: (no net) -> C10
- SW26 pad 2: (no net) -> Net-(D41-Pad2)
- SW27 pad 1: (no net) -> C11
- SW27 pad 2: (no net) -> Net-(D42-Pad2)
- SW28 pad 1: (no net) -> C12
- SW28 pad 2: (no net) -> Net-(D43-Pad2)
- SW29 pad 1: (no net) -> C13
- SW29 pad 2: (no net) -> Net-(D44-Pad2)
- SW3 pad 1: (no net) -> C2
- SW3 pad 2: (no net) -> Net-(D3-Pad2)
- SW30 pad 1: (no net) -> C14
- SW30 pad 2: (no net) -> Net-(D45-Pad2)
- SW31 pad 1: (no net) -> C15
- SW31 pad 2: (no net) -> Net-(D46-Pad2)
- SW32 pad 1: (no net) -> C0
- SW32 pad 2: (no net) -> Net-(D63-Pad2)
- SW33 pad 1: (no net) -> C1
- SW33 pad 2: (no net) -> Net-(D64-Pad2)
- SW34 pad 1: (no net) -> C2
- SW34 pad 2: (no net) -> Net-(D65-Pad2)
- SW35 pad 1: (no net) -> C3
- SW35 pad 2: (no net) -> Net-(D66-Pad2)
- SW36 pad 1: (no net) -> C4
- SW36 pad 2: (no net) -> Net-(D67-Pad2)
- SW37 pad 1: (no net) -> C5
- SW37 pad 2: (no net) -> Net-(D68-Pad2)
- SW38 pad 1: (no net) -> C6
- SW38 pad 2: (no net) -> Net-(D69-Pad2)
- SW39 pad 1: (no net) -> C7
- SW39 pad 2: (no net) -> Net-(D70-Pad2)
- SW4 pad 1: (no net) -> C3
- SW4 pad 2: (no net) -> Net-(D4-Pad2)
- SW40 pad 1: (no net) -> C8
- SW40 pad 2: (no net) -> Net-(D71-Pad2)
- SW41 pad 1: (no net) -> C9
- SW41 pad 2: (no net) -> Net-(D72-Pad2)
- SW42 pad 1: (no net) -> C10
- SW42 pad 2: (no net) -> Net-(D73-Pad2)
- SW43 pad 1: (no net) -> C11
- SW43 pad 2: (no net) -> Net-(D74-Pad2)
- SW44 pad 1: (no net) -> C12
- SW44 pad 2: (no net) -> Net-(D75-Pad2)
- SW45 pad 1: (no net) -> C13
- SW45 pad 2: (no net) -> Net-(D76-Pad2)
- SW46 pad 1: (no net) -> C14
- SW46 pad 2: (no net) -> Net-(D77-Pad2)
- SW47 pad 1: (no net) -> C15
- SW47 pad 2: (no net) -> Net-(D78-Pad2)
- SW48 pad 1: (no net) -> C0
- SW48 pad 2: (no net) -> Net-(D95-Pad2)
- SW49 pad 1: (no net) -> C1
- SW49 pad 2: (no net) -> Net-(D96-Pad2)
- SW5 pad 1: (no net) -> C4
- SW5 pad 2: (no net) -> Net-(D5-Pad2)
- SW50 pad 1: (no net) -> C2
- SW50 pad 2: (no net) -> Net-(D97-Pad2)
- SW51 pad 1: (no net) -> C3
- SW51 pad 2: (no net) -> Net-(D98-Pad2)
- SW52 pad 1: (no net) -> C4
- SW52 pad 2: (no net) -> Net-(D99-Pad2)
- SW53 pad 1: (no net) -> C5
- SW53 pad 2: (no net) -> Net-(D100-Pad2)
- SW54 pad 1: (no net) -> C6
- SW54 pad 2: (no net) -> Net-(D101-Pad2)
- SW55 pad 1: (no net) -> C7
- SW55 pad 2: (no net) -> Net-(D102-Pad2)
- SW56 pad 1: (no net) -> C8
- SW56 pad 2: (no net) -> Net-(D103-Pad2)
- SW57 pad 1: (no net) -> C9
- SW57 pad 2: (no net) -> Net-(D104-Pad2)
- SW58 pad 1: (no net) -> C10
- SW58 pad 2: (no net) -> Net-(D105-Pad2)
- SW59 pad 1: (no net) -> C11
- SW59 pad 2: (no net) -> Net-(D106-Pad2)
- SW6 pad 1: (no net) -> C5
- SW6 pad 2: (no net) -> Net-(D6-Pad2)
- SW60 pad 1: (no net) -> C12
- SW60 pad 2: (no net) -> Net-(D107-Pad2)
- SW61 pad 1: (no net) -> C13
- SW61 pad 2: (no net) -> Net-(D108-Pad2)
- SW62 pad 1: (no net) -> C14
- SW62 pad 2: (no net) -> Net-(D109-Pad2)
- SW63 pad 1: (no net) -> C15
- SW63 pad 2: (no net) -> Net-(D110-Pad2)
- SW64 pad 1: (no net) -> C0
- SW64 pad 2: (no net) -> Net-(D127-Pad2)
- SW65 pad 1: (no net) -> C1
- SW65 pad 2: (no net) -> Net-(D128-Pad2)
- SW66 pad 1: (no net) -> C2
- SW66 pad 2: (no net) -> Net-(D129-Pad2)
- SW67 pad 1: (no net) -> C3
- SW67 pad 2: (no net) -> Net-(D130-Pad2)
- SW69 pad 1: (no net) -> C5
- SW69 pad 2: (no net) -> Net-(D132-Pad2)
- SW7 pad 1: (no net) -> C6
- SW7 pad 2: (no net) -> Net-(D7-Pad2)
- SW70 pad 1: (no net) -> C6
- SW70 pad 2: (no net) -> Net-(D133-Pad2)
- SW71 pad 1: (no net) -> C7
- SW71 pad 2: (no net) -> Net-(D134-Pad2)
- SW72 pad 1: (no net) -> C8
- SW72 pad 2: (no net) -> Net-(D135-Pad2)
- SW73 pad 1: (no net) -> C9
- SW73 pad 2: (no net) -> Net-(D136-Pad2)
- SW74 pad 1: (no net) -> C10
- SW74 pad 2: (no net) -> Net-(D137-Pad2)
- SW75 pad 1: (no net) -> C11
- SW75 pad 2: (no net) -> Net-(D138-Pad2)
- SW76 pad 1: (no net) -> C12
- SW76 pad 2: (no net) -> Net-(D139-Pad2)
- SW77 pad 1: (no net) -> C13
- SW77 pad 2: (no net) -> Net-(D140-Pad2)
- SW78 pad 1: (no net) -> C14
- SW78 pad 2: (no net) -> Net-(D141-Pad2)
- SW79 pad 1: (no net) -> C15
- SW79 pad 2: (no net) -> Net-(D142-Pad2)
- SW8 pad 1: (no net) -> C7
- SW8 pad 2: (no net) -> Net-(D8-Pad2)
- SW80 pad 1: (no net) -> C0
- SW80 pad 2: (no net) -> Net-(D159-Pad2)
- SW81 pad 1: (no net) -> C1
- SW81 pad 2: (no net) -> Net-(D160-Pad2)
- SW82 pad 1: (no net) -> C2
- SW82 pad 2: (no net) -> Net-(D161-Pad2)
- SW83 pad 1: (no net) -> C3
- SW83 pad 2: (no net) -> Net-(D162-Pad2)
- SW84 pad 1: (no net) -> C4
- SW84 pad 2: (no net) -> Net-(D163-Pad2)
- SW85 pad 1: (no net) -> C5
- SW85 pad 2: (no net) -> Net-(D164-Pad2)
- SW86 pad 1: (no net) -> C6
- SW86 pad 2: (no net) -> Net-(D165-Pad2)
- SW87 pad 1: (no net) -> C7
- SW87 pad 2: (no net) -> Net-(D166-Pad2)
- SW88 pad 1: (no net) -> C8
- SW88 pad 2: (no net) -> Net-(D167-Pad2)
- SW89 pad 1: (no net) -> C9
- SW89 pad 2: (no net) -> Net-(D168-Pad2)
- SW9 pad 1: (no net) -> C8
- SW9 pad 2: (no net) -> Net-(D9-Pad2)
- SW90 pad 1: (no net) -> C10
- SW90 pad 2: (no net) -> Net-(D169-Pad2)
- SW91 pad 1: (no net) -> C11
- SW91 pad 2: (no net) -> Net-(D170-Pad2)
- SW92 pad 1: (no net) -> C12
- SW92 pad 2: (no net) -> Net-(D171-Pad2)
- SW93 pad 1: (no net) -> C13
- SW93 pad 2: (no net) -> Net-(D172-Pad2)
- SW94 pad 1: (no net) -> C14
- SW94 pad 2: (no net) -> Net-(D173-Pad2)
- SW95 pad 1: (no net) -> C15
- SW95 pad 2: (no net) -> Net-(D174-Pad2)
- SW96 pad 1: (no net) -> C0
- SW96 pad 2: (no net) -> Net-(D191-Pad2)
- SW97 pad 1: (no net) -> C1
- SW97 pad 2: (no net) -> Net-(D192-Pad2)
Other:
- outline, holes or cut-outs redrawn
- board text removed: "RCK v1.0 Jan. 2023"
- board text removed: "Raúl Reinosa Simón"

Commit message: software changes
Parts:
- removed SW1, SW10, SW11, SW12, SW13, SW14, SW15, SW16, SW17, SW18, SW19, SW2, SW20, SW21, SW22, SW23, SW24, SW25, SW26, SW27, SW28, SW3, SW30, SW31, SW32, SW33, SW35, SW36, SW37, SW38, SW39, SW4, SW40, SW41, SW42, SW43, SW44, SW45, SW46, SW48, SW49, SW5, SW50, SW53, SW54, SW55, SW56, SW57, SW58, SW59, SW6, SW60, SW61, SW62, SW63, SW64, SW65, SW66, SW67, SW69, SW7, SW70, SW71, SW72, SW73, SW74, SW75, SW76, SW77, SW78, SW79, SW8, SW80, SW81, SW82, SW83, SW84, SW87, SW88, SW9, SW90, SW91, SW93, SW94, SW95, SW96, SW97: SW_Push, Button_Switch_Keyboard:SW_Cherry_MX_1.00u_Plate
- removed SW29: SW_Push, Button_Switch_Keyboard:SW_Cherry_MX_2.00u_PCB
- removed SW34, SW86: SW_Push, Button_Switch_Keyboard:SW_Cherry_MX_1.50u_Plate
- removed SW47: SW_Push, Button_Switch_Keyboard:SW_Cherry_MX_ISOEnter_PCB
- removed SW51, SW85: SW_Push, Button_Switch_Keyboard:SW_Cherry_MX_2.00u_Vertical_PCB
- removed SW52: SW_Push, Button_Switch_Keyboard:SW_Cherry_MX_1.75u_Plate
- removed SW89: SW_Push, Button_Switch_Keyboard:SW_Cherry_MX_6.25u_PCB
- removed SW92: SW_Push, Button_Switch_Keyboard:SW_Cherry_MX_1.25u_Plate
Other:
- outline, holes or cut-outs redrawn
