File: v1.0/plate/plate.sch (KiCad schematic (older format))
At the start: 107 parts, among them SW1 SW_Push, SW10 SW_Push, SW11 SW_Push, SW12 SW_Push, SW13 SW_Push, SW14 SW_Push, SW15 SW_Push, SW16 SW_Push, SW18 SW_Push, SW19 SW_Push, SW2 SW_Push, SW20 SW_Push, SW21 SW_Push, SW22 SW_Push, SW23 SW_Push, SW24 SW_Push, SW25 SW_Push, SW26 SW_Push, SW27 SW_Push, SW28 SW_Push, SW29 SW_Push, SW3 SW_Push, SW30 SW_Push, SW31 SW_Push, SW32 SW_Push, SW33 SW_Push, SW34 SW_Push, SW35 SW_Push, SW36 SW_Push, SW37 SW_Push, SW38 SW_Push, SW39 SW_Push, SW4 SW_Push, SW40 SW_Push, SW41 SW_Push, SW42 SW_Push, SW43 SW_Push, SW44 SW_Push, SW45 SW_Push, SW46 SW_Push, SW47 SW_Push, SW48 SW_Push, SW49 SW_Push, SW5 SW_Push, SW50 SW_Push, SW51 SW_Push, SW52 SW_Push, SW53 SW_Push, SW54 SW_Push, SW55 SW_Push, SW56 SW_Push, SW57 SW_Push, SW58 SW_Push, SW59 SW_Push, SW6 SW_Push, SW60 SW_Push, SW61 SW_Push, SW62 SW_Push, SW63 SW_Push, SW64 SW_Push, SW65 SW_Push, SW66 SW_Push, SW67 SW_Push, SW68 SW_Push, SW69 SW_Push, SW7 SW_Push, SW70 SW_Push, SW71 SW_Push, SW72 SW_Push, SW73 SW_Push, SW74 SW_Push, SW75 SW_Push, SW76 SW_Push, SW77 SW_Push, SW78 SW_Push, SW79 SW_Push, SW8 SW_Push, SW80 SW_Push, SW81 SW_Push, SW82 SW_Push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

Commit message: plate
Parts:
- added C1, C2, C3, C5, C8: 0.1uF, Capacitor_SMD:C_1206_3216Metric, symbol Device:C_Small
- added C4: 10uF, Capacitor_SMD:C_1206_3216Metric, symbol Device:C_Small
- added C6, C7: 22uF, Capacitor_SMD:C_1206_3216Metric, symbol Device:C_Small
- added C9: 1uF, Capacitor_SMD:C_1206_3216Metric, symbol Device:C_Small
- added D1, D10, D100, D101, D102, D103, D104, D105, D106, D107, D108, D109, D11, D110, D12, D127, D128, D129, D13, D130, D131, D132, D133, D134, D135, D136, D137, D138, D139, D14, D140, D141, D142, D15, D159, D160, D161, D162, D163, D164, D165, D166, D167, D168, D169, D170, D171, D172, D173, D174, D191, D192, D2, D3, D31, D32, D33, D34, D35, D36, D37, D38, D39, D4, D40, D41, D42, D43, D44, D45, D46, D5, D6, D63, D64, D65, D66, D67, D68, D69, D7, D70, D71, D72, D73, D74, D75, D76, D77, D78, D8, D9, D95, D96, D97, D98, D99: 1N4148W, Diode_SMD:D_SOD-123, symbol Diode:1N4148W
- added D111, D112, D113, D114, D115, D116, D117, D118, D119, D120, D121, D122, D123, D124, D125, D126, D143, D144, D145, D146, D147, D148, D149, D150, D151, D152, D153, D154, D155, D156, D157, D158, D16, D17, D175, D176, D177, D178, D179, D18, D180, D181, D182, D183, D184, D185, D186, D187, D188, D189, D19, D190, D193, D194, D20, D21, D22, D23, D24, D25, D26, D27, D28, D29, D30, D47, D48, D49, D50, D51, D52, D53, D54, D55, D56, D57, D58, D59, D60, D61, D62, D79, D80, D81, D82, D83, D84, D85, D86, D87, D88, D89, D90, D91, D92, D93, D94: SK6812, LED_SMD:LED_SK6812_PLCC4_5.0x5.0mm_P3.2mm, symbol LED:SK6812
- added F1: 500mA, Fuse:Fuse_1206_3216Metric, symbol Device:Polyfuse
- added J1: USB_C_Receptacle_USB2.0, Connector_USB:USB_C_Receptacle_HRO_TYPE-C-31-M-12, symbol Connector:USB_C_Receptacle_USB2.0
- added J2: ISP, Connector_PinHeader_2.54mm:PinHeader_2x03_P2.54mm_Vertical, symbol Connector_Generic:Conn_02x03_Counter_Clockwise
- added R1, R5: 10k, Resistor_SMD:R_1206_3216Metric, symbol Device:R_Small
- added R2, R3, R6, R7: 22, Resistor_SMD:R_1206_3216Metric, symbol Device:R_Small
- added R4: 330, Resistor_SMD:R_1206_3216Metric, symbol Device:R_Small
- added U1: CD74HC4067M, Package_SO:SOIC-24W_7.5x15.4mm_P1.27mm, symbol 74xx:CD74HC4067M
- added U2: ATmega32U4-AU, Package_QFP:TQFP-44_10x10mm_P0.8mm, symbol MCU_Microchip_ATmega:ATmega32U4-AU
- added Y1: 16MHz, Crystal:Crystal_SMD_HC49-SD, symbol Device:Crystal_Small
- renumbered SW18 to SW16, SW19 to SW17, SW20 to SW18, SW21 to SW19, SW22 to SW20, SW23 to SW21, SW24 to SW22, SW25 to SW23, SW26 to SW24, SW27 to SW25, SW28 to SW26, SW29 to SW27, SW30 to SW28, SW31 to SW29, SW32 to SW30, SW33 to SW31, SW34 to SW32, SW35 to SW33, SW36 to SW34, SW37 to SW35, SW38 to SW36, SW39 to SW37, SW40 to SW38, SW41 to SW39, SW42 to SW40, SW43 to SW41, SW44 to SW42, SW45 to SW43, SW46 to SW44, SW47 to SW45, SW48 to SW46, SW49 to SW47, SW50 to SW48, SW51 to SW49, SW52 to SW50, SW53 to SW51, SW54 to SW52, SW55 to SW53, SW56 to SW54, SW57 to SW55, SW58 to SW56, SW59 to SW57, SW60 to SW58, SW61 to SW59, SW62 to SW60, SW63 to SW61, SW64 to SW62, SW65 to SW63, SW66 to SW64, SW67 to SW65, SW68 to SW66, SW69 to SW67, SW70 to SW68, SW71 to SW69, SW72 to SW70, SW73 to SW71, SW74 to SW72, SW75 to SW73, SW76 to SW74, SW77 to SW75, SW78 to SW76, SW79 to SW77, SW80 to SW78, SW81 to SW79, SW82 to SW80, SW83 to SW81, SW84 to SW82, SW85 to SW83, SW86 to SW84, SW87 to SW85, SW88 to SW86, SW89 to SW87, SW90 to SW88, SW91 to SW89, SW92 to SW90, SW93 to SW91, SW94 to SW92, SW95 to SW93, SW96 to SW94, SW97 to SW95, SW98 to SW96, SW16 to SW97
Connections:
- net labels added: +5V, COM, D+, D-, LED0, LED1, LED2, LED3, LED4, LED5, LED6, MISO, MOSI, R0, R1, R2, R3, R4, R5, R6, S0, S1, S2, S3, SCK, SE
- wire segments 34 -> 686
- no-connect marks 2 -> 16

Commit message: plate done
Parts:
- removed C1, C2, C3, C5, C8: 0.1uF, Capacitor_SMD:C_1206_3216Metric, symbol Device:C_Small
- removed C4: 10uF, Capacitor_SMD:C_1206_3216Metric, symbol Device:C_Small
- removed C6, C7: 22uF, Capacitor_SMD:C_1206_3216Metric, symbol Device:C_Small
- removed C9: 1uF, Capacitor_SMD:C_1206_3216Metric, symbol Device:C_Small
- removed F1: 500mA, Fuse:Fuse_1206_3216Metric, symbol Device:Polyfuse
- removed J1: USB_C_Receptacle_USB2.0, Connector_USB:USB_C_Receptacle_HRO_TYPE-C-31-M-12, symbol Connector:USB_C_Receptacle_USB2.0
- removed J2: ISP, Connector_PinHeader_2.54mm:PinHeader_2x03_P2.54mm_Vertical, symbol Connector_Generic:Conn_02x03_Counter_Clockwise
- removed R1, R5: 10k, Resistor_SMD:R_1206_3216Metric, symbol Device:R_Small
- removed R2, R3, R6, R7: 22, Resistor_SMD:R_1206_3216Metric, symbol Device:R_Small
- removed U1: CD74HC4067M, Package_SO:SOIC-24W_7.5x15.4mm_P1.27mm, symbol 74xx:CD74HC4067M
- removed U2: ATmega32U4-AU, Package_QFP:TQFP-44_10x10mm_P0.8mm, symbol MCU_Microchip_ATmega:ATmega32U4-AU
- removed Y1: 16MHz, Crystal:Crystal_SMD_HC49-SD, symbol Device:Crystal_Small
Connections:
- net labels removed: COM, D+, D-, MISO, MOSI, S0, S1, S2, S3, SCK, SE
- wire segments 686 -> 608
- no-connect marks 16 -> 3
