File: v0.1/pcb/pcb.kicad_pcb (KiCad board)
At the start: 2 copper layers, 50 x 50 mm, 30 parts, among them J1 USB_C_Receptacle_USB2.0, J2 ISP, SW1 SW_Push, SW2 SW_Push, U1 ATmega32U4-AU, Y1 16MHz

Commit message: create new gerbers files
Parts:
- removed R3, R6: 22, Resistor_SMD:R_1206_3216Metric
- removed R7: 10k, Resistor_SMD:R_1206_3216Metric
- C5, C6: value 22uF -> 22pF
- C7: value 100nF -> 0.1uF
Connections:
- J2 pad 3: (no net) -> RST
- R4 pad 2: Net-(R4-Pad2) -> RST
- U1 pad 13: Net-(R4-Pad2) -> RST
- U1 pad 18: (no net) -> LED0
- U1 pad 3: Net-(R6-Pad1) -> D-
- U1 pad 33: Net-(R7-Pad2) -> GND
- U1 pad 38: LED0 -> (no net)
- U1 pad 4: Net-(R3-Pad1) -> D+
Routing:
- net RST: track 0.00 -> 48.3 mm, vias 0 -> 4
- net D+: track 2.41 -> 33.0 mm, vias 0 -> 4
- net Net-(R3-Pad1): track 27.7 -> 0.00 mm, vias 2 -> 0
- net Net-(R4-Pad2): track 24.9 -> 0.00 mm, vias 2 -> 0
- net D-: track 2.41 -> 20.2 mm, vias 0 -> 2
- net Net-(R6-Pad1): track 15.0 -> 0.00 mm, vias 2 -> 0
- net Net-(R7-Pad2): track 14.2 -> 0.00 mm, vias 2 -> 0
- net GND: track 11.0 -> 25.2 mm, vias 6 -> 9
- net LED0: track 48.8 -> 44.1 mm, vias 0 -> 4
- net +5V: track 127.7 -> 131.0 mm
- net MOSI: track 31.0 -> 33.1 mm
- net Net-(D3-Pad2): track 22.6 -> 24.2 mm
- net Net-(C6-Pad2): track 44.2 -> 45.4 mm
