File: v0.1/pcb/pcb.sch (KiCad schematic (older format))
At the start: 30 parts, among them J1 USB_C_Receptacle_USB2.0, J2 ISP, SW1 SW_Push, SW2 SW_Push, U1 ATmega32U4-AU, Y1 16MHz

Commit message: updating software features
Parts:
- removed R3, R6: 22, Resistor_SMD:R_1206_3216Metric, symbol Device:R_Small
- removed R7: 10k, Resistor_SMD:R_1206_3216Metric, symbol Device:R_Small
- C5, C6: value 22uF -> 22pF
Connections:
- net D+: now also U1.4 (D+)
- net D-: now also U1.3 (D-)
- net GND: now also U1.33 (~HWB~/PE2)
- net RST: now reaches R4.2, U1.13 (~RESET)
- net RST: now also J2.3 (Pin_3)
- no-connect marks 26 -> 25
Changed lines of the file:
@@
 EESchema Schematic File Version 4
-LIBS:test-cache
+LIBS:pcb-cache
 EELAYER 30 0
 EELAYER END
@@
 NoConn ~ 2000 -600
 NoConn ~ 3500 11650
-$Comp
-L Connector_Generic:Conn_02x03_Counter_Clockwise J2
-U 1 1 676CACE0
-P 3150 6800
-F 0 "J2" H 3200 7117 50  0000 C CNN
-F 1 "ISP" H 3200 7026 50  0000 C CNN
-F 2 "Connector_PinHeader_2.54mm:PinHeader_2x03_P2.54mm_Vertical" H 3150 6800 50  0001 C CNN
-F 3 "~" H 3150 6800 50  0001 C CNN
-	1    3150 6800
-	1    0    0    -1
-$EndComp
 Text GLabel 2950 6700 0    50   Input ~ 0
 MISO
@@
 R0
 $Comp
-L Device:R_Small R7
-U 1 1 63D596F6
-P 4200 4550
-F 0 "R7" V 4004 4550 50  0000 C CNN
-F 1 "10k" V 4095 4550 50  0000 C CNN
-F 2 "Resistor_SMD:R_1206_3216Metric" H 4200 4550 50  0001 C CNN
-F 3 "~" H 4200 4550 50  0001 C CNN
-	1    4200 4550
-	0    1    1    0
-$EndComp
-$Comp
 L power:GND #PWR09
 U 1 1 63D5B1DE
@@
 	1    0    0    -1
 $EndComp
-Wire Wire Line
-	4300 4550 4550 4550
-$Comp
-L Device:R_Small R3
-U 1 1 63D5D756
-P 2100 3450
-F 0 "R3" V 1904 3450 50  0000 C CNN
-F 1 "22" V 1995 3450 50  0000 C CNN
-F 2 "Resistor_SMD:R_1206_3216Metric" H 2100 3450 50  0001 C CNN
-F 3 "~" H 2100 3450 50  0001 C CNN
-	1    2100 3450
-	0    1    1    0
-$EndComp
-$Comp
-L Device:R_Small R6
-U 1 1 63D5DFD0
-P 2100 3550
-F 0 "R6" V 2200 3550 50  0000 C CNN
-F 1 "22" V 2300 3550 50  0000 C CNN
-F 2 "Resistor_SMD:R_1206_3216Metric" H 2100 3550 50  0001 C CNN
-F 3 "~" H 2100 3550 50  0001 C CNN
-	1    2100 3550
-	0    1    1    0
-$EndComp
 $Comp
 L power:GND #PWR07
@@
 P 1750 2900
 F 0 "C6" V 1650 3000 50  0000 C CNN
-F 1 "22uF" V 1650 2750 50  0000 C CNN
+F 1 "22pF" V 1650 2750 50  0000 C CNN
 F 2 "Capacitor_SMD:C_1206_3216Metric" H 1750 2900 50  0001 C CNN
 F 3 "~" H 1750 2900 50  0001 C CNN
@@
 Wire Wire Line
 	3450 1900 3850 1900
-Wire Wire Line
-	3750 4550 4100 4550
 $Comp
 L power:GND #PWR011
@@
 	1    0    0    -1
 $EndComp
-$Comp
-L MCU_Microchip_ATmega:ATmega32U4-AU U1
-U 1 1 63D52C27
-P 3150 3950
-F 0 "U1" V 2450 2600 50  0000 C CNN
-F 1 "ATmega32U4-AU" V 2550 2600 50  0000 C CNN
-F 2 "Package_QFP:TQFP-44_10x10mm_P0.8mm" H 3150 3950 50  0001 C CIN
-F 3 "http://ww1.microchip.com/downloads/en/DeviceDoc/Atmel-7766-8-bit-AVR-ATmega16U4-32U4_Datasheet.pdf" H 3150 3950 50  0001 C CNN
-	1    3150 3950
-	1    0    0    -1
-$EndComp
 Wire Wire Line
 	2500 2450 2500 2150
@@
 Wire Wire Line
 	2500 1750 3050 1750
-Wire Wire Line
-	2550 3550 2200 3550
-Wire Wire Line
-	2550 3450 2200 3450
-Wire Wire Line
-	1850 3450 2000 3450
-Wire Wire Line
-	2000 3550 1850 3550
 Wire Wire Line
 	2550 3750 2250 3750
@@
 P 1750 2550
 F 0 "C5" V 2000 2550 50  0000 C CNN
-F 1 "22uF" V 1900 2550 50  0000 C CNN
+F 1 "22pF" V 1900 2550 50  0000 C CNN
 F 2 "Capacitor_SMD:C_1206_3216Metric" H 1750 2550 50  0001 C CNN
 F 3 "~" H 1750 2550 50  0001 C CNN
@@
 Wire Wire Line
 	2150 3050 2550 3050
-NoConn ~ 2950 6900
 Wire Wire Line
 	7300 2400 7300 2450
@@
 Wire Wire Line
 	2550 3250 2250 3250
+$Comp
+L MCU_Microchip_ATmega:ATmega32U4-AU U1
+U 1 1 63D52C27
+P 3150 3950
+F 0 "U1" V 2450 2600 50  0000 C CNN
+F 1 "ATmega32U4-AU" V 2550 2600 50  0000 C CNN
+F 2 "Package_QFP:TQFP-44_10x10mm_P0.8mm" H 3150 3950 50  0001 C CIN
+F 3 "http://ww1.microchip.com/downloads/en/DeviceDoc/Atmel-7766-8-bit-AVR-ATmega16U4-32U4_Datasheet.pdf" H 3150 3950 50  0001 C CNN
+	1    3150 3950
+	1    0    0    -1
+$EndComp
+Wire Wire Line
+	3750 4550 4550 4550
+Wire Wire Line
+	1850 3550 2550 3550
+Wire Wire Line
+	1850 3450 2550 3450
+$Comp
+L Connector_Generic:Conn_02x03_Counter_Clockwise J2
+U 1 1 676CACE0
+P 3150 6800
+F 0 "J2" H 3200 7117 50  0000 C CNN
+F 1 "ISP" H 3200 7026 50  0000 C CNN
+F 2 "Connector_PinHeader_2.54mm:PinHeader_2x03_P2.54mm_Vertical" H 3150 6800 50  0001 C CNN
+F 3 "~" H 3150 6800 50  0001 C CNN
+	1    3150 6800
+	1    0    0    -1
+$EndComp
+Text GLabel 2950 6900 0    50   Input ~ 0
+RST
+Text GLabel 2400 2450 0    50   Input ~ 0
+RST
+Wire Wire Line
+	2500 2450 2400 2450
+Connection ~ 2500 2450
 $EndSCHEMATC

Commit message: create new gerbers files
Connections:
- net LED0: now also U1.18 (PD0); no longer U1.38 (PF5)
Changed lines of the file:
@@
 NoConn ~ 3750 3850
 NoConn ~ 3750 3750
-Text GLabel 3750 5150 2    50   Input ~ 0
+Text GLabel 3750 3650 2    50   Input ~ 0
 LED0
 Text GLabel 3750 2750 2    50   Input ~ 0
@@
 NoConn ~ 3750 5350
 NoConn ~ 3750 4350
-NoConn ~ 3750 3650
 NoConn ~ 3750 2850
 NoConn ~ 3750 3350
 Wire Wire Line
 	2550 3250 2250 3250
+Wire Wire Line
+	3750 4550 4550 4550
+Wire Wire Line
+	1850 3550 2550 3550
+Wire Wire Line
+	1850 3450 2550 3450
+$Comp
+L Connector_Generic:Conn_02x03_Counter_Clockwise J2
+U 1 1 676CACE0
+P 3150 6800
+F 0 "J2" H 3200 7117 50  0000 C CNN
+F 1 "ISP" H 3200 7026 50  0000 C CNN
+F 2 "Connector_PinHeader_2.54mm:PinHeader_2x03_P2.54mm_Vertical" H 3150 6800 50  0001 C CNN
+F 3 "~" H 3150 6800 50  0001 C CNN
+	1    3150 6800
+	1    0    0    -1
+$EndComp
+Text GLabel 2950 6900 0    50   Input ~ 0
+RST
+Text GLabel 2400 2450 0    50   Input ~ 0
+RST
+Wire Wire Line
+	2500 2450 2400 2450
+Connection ~ 2500 2450
 $Comp
 L MCU_Microchip_ATmega:ATmega32U4-AU U1
@@
 	1    0    0    -1
 $EndComp
-Wire Wire Line
-	3750 4550 4550 4550
-Wire Wire Line
-	1850 3550 2550 3550
-Wire Wire Line
-	1850 3450 2550 3450
-$Comp
-L Connector_Generic:Conn_02x03_Counter_Clockwise J2
-U 1 1 676CACE0
-P 3150 6800
-F 0 "J2" H 3200 7117 50  0000 C CNN
-F 1 "ISP" H 3200 7026 50  0000 C CNN
-F 2 "Connector_PinHeader_2.54mm:PinHeader_2x03_P2.54mm_Vertical" H 3150 6800 50  0001 C CNN
-F 3 "~" H 3150 6800 50  0001 C CNN
-	1    3150 6800
-	1    0    0    -1
-$EndComp
-Text GLabel 2950 6900 0    50   Input ~ 0
-RST
-Text GLabel 2400 2450 0    50   Input ~ 0
-RST
-Wire Wire Line
-	2500 2450 2400 2450
-Connection ~ 2500 2450
+NoConn ~ 3750 5150
 $EndSCHEMATC
